File: pouch2/pouch2.kicad_pcb (KiCad board)
At the start: 2 copper layers, 75 x 100 mm, 93 parts, among them J101 Conn_01x04_Male, J102 Conn_01x06_Male, J103 Conn_01x03_Male, J501 Conn_01x02_Male, J502 Conn_01x02_Male, J503 Conn_01x02_Male, J504 Conn_01x02_Male, J701 Conn_01x14_Male, J702 Conn_01x14_Male, J703 Conn_01x14_Male, J704 Conn_01x14_Male, J705 Conn_01x14_Male, J706 Conn_01x14_Male, J707 Conn_01x14_Male, J708 Conn_01x14_Male, J801 PiZero, K801 AZ9371-1A-5DE, Q501 AO3401A, Q502 AO3401A, Q503 AO3401A, Q504 AO3401A, Q801 MMBT3906, SW501 SW_SPDT, SW701 SW_DIP_x08, U101 Pico, U201 BME688, U202 BME280

Commit message: PCB and footprint arrangements
Parts:
- added G***: LOGO, LOGO, F.Cu at (128.0, 178.5)
- added H101: MountingHole, MountingHole:MountingHole_3.2mm_M3_DIN965_Pad_TopBottom, F.Cu at (55.0, 55.0)
- added H102: MountingHole, MountingHole:MountingHole_3.2mm_M3_DIN965_Pad_TopBottom, F.Cu at (125.0, 55.0)
- added H103: MountingHole, MountingHole:MountingHole_3.2mm_M3_DIN965_Pad_TopBottom, F.Cu at (55.0, 145.0)
- added H104: MountingHole, MountingHole:MountingHole_3.2mm_M3_DIN965_Pad_TopBottom, F.Cu at (125.0, 145.0)
- BT501: footprint Battery:BatteryHolder_Keystone_1042_1x18650 -> SensorBoards:18650_Keystone_1043
- J801: footprint Module:Raspberry_Pi_Zero_Socketed_THT_FaceDown_MountingHoles -> SensorBoards:Raspberry_Pi_Zero_Socket_wo_drills
- SW701: footprint Package_DIP:DIP-16_W7.62mm -> Button_Switch_THT:SW_DIP_SPSTx08_Slide_9.78x22.5mm_W7.62mm_P2.54mm
- moved BT501 228.0 mm to (90.0, 72.5)
- moved J701 224.6 mm to (235.5, 132.1), turned to 90 degrees
- moved J702 220.0 mm to (235.5, 129.5), turned to 90 degrees
- moved J703 215.4 mm to (235.5, 127.0), turned to 90 degrees
- moved J704 210.9 mm to (235.5, 124.5), turned to 90 degrees
- moved D801 210.1 mm to (212.7, 125.7)
- moved J101 210.1 mm to (181.3, 129.1)
- moved J504 210.1 mm to (166.5, 94.6)
- moved Q801 210.1 mm to (208.0, 126.4)
- moved R207 210.1 mm to (269.6, 81.7)
- moved R208 210.1 mm to (269.6, 84.7)
- moved R209 210.1 mm to (269.6, 87.6)
- moved R801 210.1 mm to (203.4, 125.7)
- moved R802 210.1 mm to (203.4, 128.6)
- moved R803 210.1 mm to (203.4, 131.6)
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Connections:
- J708 pad 14: unconnected-(J708-Pin_14-Pad14) -> -BATT
Other:
- board size 75 x 100 mm -> 80 x 100 mm
- board text added: "A]"
- board text added: "B]"
- board text added: "Campaign ID"
- board text added: "DTAC TP2 - pouch2 Leon Schnieber Bernhard Lehner"

Commit message: updated backside of PCB
Parts:
- added XX201: DEBO_MPU-6050, SensorBoards:DEBO_MPU6050, F.Cu at (123.2, 126.2)
- D801, JP201, JP202, JP203, Q501, Q502, Q503, Q504, Q801, R101, R102, R103, R104, R105, R106, R107, R108, R109, R110, R111, R112, R113, R114, R115, R116, R117, R118, R119, R120, R201, R202, R203, R204, R205, R206, R207, R208, R209, R301, R302, R303, R501, R502, R503, R504, R505, R506, R507, R508, R509, R701, R702, R703, R704, R705, R706, R707, R708, R801, R802, R803, R804, R805, U101, U201, U202: moved to B.Cu
- U301: footprint Connector_PinHeader_2.54mm:PinHeader_1x09_P2.54mm_Vertical -> SensorBoards:DEBO_GPS
- U401: footprint Connector_PinHeader_2.54mm:PinHeader_1x06_P2.54mm_Vertical -> SensorBoards:DEBO_SD-Card
- moved R301 220.0 mm to (42.5, 150.3), turned to 180 degrees
- moved R302 220.0 mm to (42.5, 153.2), turned to 180 degrees
- moved R303 220.0 mm to (42.5, 156.2), turned to 180 degrees
- moved R708 201.4 mm to (88.7, 53.2), turned to 180 degrees
- moved R707 200.4 mm to (87.3, 56.2), turned to 90 degrees
- moved R706 197.4 mm to (89.4, 56.2), turned to 90 degrees
- moved R705 193.9 mm to (92.0, 56.1), turned to 90 degrees
- moved U601 190.1 mm to (77.2, 141.2), turned to 90 degrees
- moved R704 190.1 mm to (94.9, 56.2), turned to 90 degrees
- moved U401 188.9 mm to (88.2, 90.7)
- moved R701 180.8 mm to (102.8, 53.0)
- moved R702 174.9 mm to (110.1, 53.0)
- moved R703 169.1 mm to (117.6, 53.1)
- moved R507 166.5 mm to (24.3, 72.2), turned to 180 degrees
- moved R508 166.5 mm to (24.3, 75.2), turned to 180 degrees
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Connections:
- J701 pad 1: +3.3V -> -BATT
- J701 pad 14: -BATT -> +3.3V
- J702 pad 1: +3.3V -> -BATT
- J702 pad 14: -BATT -> +3.3V
- J703 pad 1: +3.3V -> -BATT
- J703 pad 14: -BATT -> +3.3V
- J704 pad 1: +3.3V -> -BATT
- J704 pad 14: -BATT -> +3.3V
- J705 pad 1: +3.3V -> -BATT
- J705 pad 14: -BATT -> +3.3V
- J706 pad 1: +3.3V -> -BATT
- J706 pad 14: -BATT -> +3.3V
- J707 pad 1: +3.3V -> -BATT
- J707 pad 14: -BATT -> +3.3V
- J708 pad 1: +3.3V -> -BATT
- J708 pad 14: -BATT -> +3.3V
Other:
- board text added: "(BME280)"
- board text added: "(BME688)"
- board text added: "(MPU6050)"
- board text added: "J102=GPS U601=eInk"
- board text added: "RX TX ⏚"
- board text added: "VCC SCL SDA ⏚"
- board text added: "⏚ PPS FIX RX TX"

Commit message: started routing
Parts:
- added JP501: Jumper_2_Open, Jumper:SolderJumper-2_P1.3mm_Open_TrianglePad1.0x1.5mm, B.Cu at (77.2, 61.9)
- added JP502: Jumper_2_Open, Jumper:SolderJumper-2_P1.3mm_Open_TrianglePad1.0x1.5mm, B.Cu at (74.7, 62.0)
- added JP503: Jumper_2_Bridged, Jumper:SolderJumper-2_P1.3mm_Bridged2Bar_Pad1.0x1.5mm, B.Cu at (57.4, 73.0)
- added R121: 0, Resistor_SMD:R_0805_2012Metric, B.Cu at (157.3, 98.2)
- added R304: 0, Resistor_SMD:R_0805_2012Metric, B.Cu at (112.7, 92.2)
- added R305: 0, Resistor_SMD:R_0805_2012Metric, B.Cu at (112.7, 95.1)
- added R401: 0, Resistor_SMD:R_0805_2012Metric, B.Cu at (163.7, 90.3)
- added R402: 0, Resistor_SMD:R_0805_2012Metric, B.Cu at (163.7, 93.3)
- added R403: 0, Resistor_SMD:R_0805_2012Metric, B.Cu at (163.7, 96.2)
- added R404: 0, Resistor_SMD:R_0805_2012Metric, B.Cu at (163.7, 99.2)
- added R601: 0, Resistor_SMD:R_0805_2012Metric, B.Cu at (170.1, 90.3)
- added R602: 0, Resistor_SMD:R_0805_2012Metric, B.Cu at (170.1, 93.3)
- added R603: 0, Resistor_SMD:R_0805_2012Metric, B.Cu at (170.1, 96.2)
- added R604: 0, Resistor_SMD:R_0805_2012Metric, B.Cu at (170.1, 99.2)
- added R605: 0, Resistor_SMD:R_0805_2012Metric, B.Cu at (170.1, 102.2)
- added R606: 0, Resistor_SMD:R_0805_2012Metric, B.Cu at (170.1, 105.1)
- added U901: SIM868, SIM868:XCVR_SIM868, B.Cu at (69.8, 97.0)
- J102: footprint Connector_PinHeader_2.54mm:PinHeader_1x06_P2.54mm_Vertical -> Connector_PinHeader_2.54mm:PinHeader_1x05_P2.54mm_Vertical
- R509: value R -> 0
- moved R301 86.3 mm to (107.8, 94.0)
- moved R302 86.3 mm to (107.8, 96.9)
- moved R303 86.3 mm to (107.8, 99.8)
- moved R110 75.8 mm to (110.5, 117.2)
- moved R102 75.6 mm to (110.6, 119.3)
- moved R115 71.1 mm to (103.2, 142.2), turned to -90 degrees
- moved R112 69.7 mm to (110.5, 113.2)
- moved R805 69.6 mm to (127.5, 114.0), turned to 0 degrees
- moved R804 69.0 mm to (127.4, 112.0), turned to 180 degrees
- moved R116 68.9 mm to (100.5, 143.2)
- moved R111 67.7 mm to (110.5, 115.2)
- moved R104 58.2 mm to (147.3, 102.2)
- moved R109 58.2 mm to (142.9, 102.2)
- moved R114 58.2 mm to (138.5, 102.2)
- moved R117 58.2 mm to (134.1, 96.3)
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Connections:
- net /SCL_PI renamed /PI_I2C0_SCL
- net /SDA_PI renamed /PI_I2C0_SDA
- net /UART_RX_PI renamed /PI_UART0_RX
- net /UART_TX_PI renamed /PI_UART0_TX
- net Net-(U101-GPIO16) renamed /PI_SPI0_RX
- net Net-(U101-GPIO17) renamed /PI_SPI0_CS
- net Net-(U101-GPIO18) renamed /PI_SPI0_SCK
- net Net-(U101-GPIO19) renamed /PI_SPI0_TX
- BT501 pad 2: -BATT -> Net-(BT501--)
- D701 pad 1: -BATT -> GND
- D702 pad 1: -BATT -> GND
- D703 pad 1: -BATT -> GND
- D801 pad 2: -BATT -> GND
- J101 pad 1: -BATT -> GND
- J102 pad 1: -BATT -> GND
- J102 pad 2: /GPS/PPS -> /UART_TX
- J102 pad 3: /GPS/FIX -> /UART_RX
- J102 pad 4: /UART_RX -> /GPS_FIX
- J102 pad 5: /UART_TX -> /GPS_PPS
- J103 pad 1: -BATT -> GND
- J701 pad 1: -BATT -> GND
- J702 pad 1: -BATT -> GND
- J703 pad 1: -BATT -> GND
- J704 pad 1: -BATT -> GND
- J705 pad 1: -BATT -> GND
- J706 pad 1: -BATT -> GND
- J707 pad 1: -BATT -> GND
- J708 pad 1: -BATT -> GND
- J801 pad 14: -BATT -> GND
- J801 pad 20: -BATT -> GND
- J801 pad 25: -BATT -> GND
- J801 pad 30: -BATT -> GND
- J801 pad 34: -BATT -> GND
- J801 pad 39: -BATT -> GND
- J801 pad 6: -BATT -> GND
- J801 pad 9: -BATT -> GND
- JP201 pad 1: -BATT -> GND
- JP202 pad 1: -BATT -> GND
- JP203 pad 1: -BATT -> GND
- K801 pad 11: /PiCoupler/PI_VCC -> +3.3V
- K801 pad A2: -BATT -> GND
- R101 pad 1: /SPI2_RST -> /DISP_RST
- R102 pad 1: /SPI2_DC -> /DISP_DC
- R103 pad 1: /SPI2_BUSY -> /DISP_BUSY
- R116 pad 2: -BATT -> GND
- R119 pad 2: /SPI_CS -> /SPI_CS_SD
- R202 pad 1: Net-(U201-SDO) -> Net-(JP202-C)
- R202 pad 2: Net-(JP202-C) -> Net-(U201-SDO)
- R203 pad 1: /SCL -> Net-(U202-SCK)
- R203 pad 2: Net-(U202-SCK) -> /SCL
- R708 pad 2: -BATT -> GND
- R803 pad 2: -BATT -> GND
- R804 pad 1: /PiCoupler/SCL -> /SCL
- R805 pad 2: /PiCoupler/SDA -> /SDA
- SW701 pad 10: unconnected-(SW701-Pad10) -> HMI_S34
- SW701 pad 11: unconnected-(SW701-Pad11) -> HMI_S24
- SW701 pad 12: unconnected-(SW701-Pad12) -> HMI_S14
- SW701 pad 5: unconnected-(SW701-Pad5) -> HMI_S13
- SW701 pad 6: unconnected-(SW701-Pad6) -> HMI_S23
- SW701 pad 7: unconnected-(SW701-Pad7) -> HMI_S33
- SW701 pad 8: unconnected-(SW701-Pad8) -> HMI_S43
- SW701 pad 9: unconnected-(SW701-Pad9) -> HMI_S44
- U101 pad 13: -BATT -> GND
- U101 pad 18: -BATT -> GND
- U101 pad 23: -BATT -> GND
- U101 pad 28: -BATT -> GND
- U101 pad 3: -BATT -> GND
- U101 pad 33: -BATT -> GND
- U101 pad 36: +3.3V -> Net-(U101-3V3)
- U101 pad 38: -BATT -> GND
- U101 pad 42: -BATT -> GND
- U101 pad 8: -BATT -> GND
- U201 pad 1: -BATT -> GND
- U201 pad 7: -BATT -> GND
- U202 pad 1: -BATT -> GND
- U202 pad 7: -BATT -> GND
- U301 pad 4: /GPS/FIX -> Net-(U301-FIX)
- U301 pad 7: -BATT -> GND
- U301 pad 9: /GPS/PPS -> Net-(U301-PPS)
- U401 pad 1: -BATT -> GND
- U401 pad 3: /SPI_RX -> Net-(U401-MISO)
- U401 pad 4: /SPI_TX -> Net-(U401-MOSI)
- U401 pad 5: /SPI_SCK -> Net-(U401-SCK)
- U401 pad 6: /SPI_CS -> Net-(U401-CS)
- U601 pad 1: /SPI2_BUSY -> Net-(U601-BUSY)
- U601 pad 2: /SPI2_DC -> Net-(U601-RST)
- U601 pad 3: /SPI2_RST -> Net-(U601-DC)
- U601 pad 4: /SPI2_CS -> Net-(U601-CS)
- U601 pad 5: /SPI2_SCK -> Net-(U601-CLK)
- U601 pad 6: /SPI2_TX -> Net-(U601-DIN)
- U601 pad 7: -BATT -> GND
- XX201 pad 2: -BATT -> GND
Routing:
- net +BATT: track 0.00 -> 94.8 mm, vias 0 -> 1
- net Net-(JP501-A): track 0.00 -> 92.0 mm, vias 0 -> 1
- net Net-(J801-Pin_3): track 0.00 -> 88.2 mm
- net Net-(J801-Pin_5): track 0.00 -> 83.3 mm
- net /PI_I2C0_SDA: track 0.00 -> 57.8 mm, vias 0 -> 2
- net /PI_I2C0_SCL: track 0.00 -> 55.6 mm, vias 0 -> 2
- net /PiCoupler/PIZERO_VCC: track 0.00 -> 46.2 mm
- net Net-(BT501-+): track 0.00 -> 35.5 mm
- net Net-(U201-SCK): track 0.00 -> 21.7 mm
- net Net-(U101-GPIO12): track 0.00 -> 21.1 mm
- net Net-(K801-Pad14): track 0.00 -> 20.4 mm, vias 0 -> 1
- net /SCL: track 0.00 -> 19.6 mm
- net /SDA: track 0.00 -> 19.4 mm
- net Net-(U201-SDI): track 0.00 -> 19.3 mm
- net Net-(U101-GPIO13): track 0.00 -> 17.6 mm
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Other:
- board text added: "⏚ TX RX FIX PPS"
- board text removed: "⏚ PPS FIX RX TX"

Commit message: drawed a lot of things
Parts:
- added R510: 0, Resistor_SMD:R_0805_2012Metric, B.Cu at (69.4, 89.4)
- added R511: 0, Resistor_SMD:R_0805_2012Metric, B.Cu at (72.8, 89.4)
- added R512: 0, Resistor_SMD:R_0805_2012Metric, B.Cu at (79.6, 89.4)
- added R513: 0, Resistor_SMD:R_0805_2012Metric, B.Cu at (76.2, 89.4)
- added R514: 0, Resistor_SMD:R_0805_2012Metric, B.Cu at (79.6, 93.4)
- added R515: 0, Resistor_SMD:R_0805_2012Metric, B.Cu at (76.2, 93.4)
- added R516: 0, Resistor_SMD:R_0805_2012Metric, B.Cu at (72.8, 93.4)
- added R517: 0, Resistor_SMD:R_0805_2012Metric, B.Cu at (69.4, 93.4)
- added R518: 0, Resistor_SMD:R_0805_2012Metric, B.Cu at (79.6, 97.4)
- added R519: 0, Resistor_SMD:R_0805_2012Metric, B.Cu at (76.2, 97.4)
- added R520: 0, Resistor_SMD:R_0805_2012Metric, B.Cu at (72.8, 97.4)
- added R521: 0, Resistor_SMD:R_0805_2012Metric, B.Cu at (69.4, 97.4)
- added R522: 0, Resistor_SMD:R_0805_2012Metric, B.Cu at (79.6, 101.4)
- added R523: 0, Resistor_SMD:R_0805_2012Metric, B.Cu at (76.2, 101.4)
- added R524: 0, Resistor_SMD:R_0805_2012Metric, B.Cu at (72.8, 101.4)
- added R525: 0, Resistor_SMD:R_0805_2012Metric, B.Cu at (69.4, 101.4)
- added R526: 0, Resistor_SMD:R_0805_2012Metric, B.Cu at (79.6, 91.4)
- added R527: 0, Resistor_SMD:R_0805_2012Metric, B.Cu at (79.6, 95.4)
- added R528: 0, Resistor_SMD:R_0805_2012Metric, B.Cu at (79.6, 99.4)
- added R529: 0, Resistor_SMD:R_0805_2012Metric, B.Cu at (79.6, 103.4)
- added R530: 0, Resistor_SMD:R_0805_2012Metric, B.Cu at (76.2, 91.4)
- added R531: 0, Resistor_SMD:R_0805_2012Metric, B.Cu at (76.2, 95.4)
- added R532: 0, Resistor_SMD:R_0805_2012Metric, B.Cu at (76.2, 99.4)
- added R533: 0, Resistor_SMD:R_0805_2012Metric, B.Cu at (76.2, 103.4)
- added R534: 0, Resistor_SMD:R_0805_2012Metric, B.Cu at (72.8, 91.4)
- added R535: 0, Resistor_SMD:R_0805_2012Metric, B.Cu at (72.8, 95.4)
- added R536: 0, Resistor_SMD:R_0805_2012Metric, B.Cu at (72.8, 99.4)
- added R537: 0, Resistor_SMD:R_0805_2012Metric, B.Cu at (72.8, 103.4)
- added R538: 0, Resistor_SMD:R_0805_2012Metric, B.Cu at (69.4, 91.4)
- added R539: 0, Resistor_SMD:R_0805_2012Metric, B.Cu at (69.4, 95.4)
- added R540: 0, Resistor_SMD:R_0805_2012Metric, B.Cu at (69.4, 99.4)
- added R541: 0, Resistor_SMD:R_0805_2012Metric, B.Cu at (69.4, 103.4)
- added R703: 0, Resistor_SMD:R_0805_2012Metric, B.Cu at (114.3, 132.0)
- added R809: 0, Resistor_SMD:R_0805_2012Metric, B.Cu at (75.1, 139.3)
- moved R114 103.8 mm to (61.4, 138.0), turned to 0 degrees
- moved U901 97.2 mm to (160.3, 61.5)
- moved R509 96.5 mm to (117.3, 103.6)
- moved R113 92.8 mm to (55.5, 140.8)
- moved R115 81.6 mm to (65.2, 138.0)
- moved R404 79.2 mm to (84.9, 90.8), turned to 0 degrees
- moved R401 79.1 mm to (84.9, 96.8)
- moved R402 78.9 mm to (84.9, 92.8)
- moved R403 78.8 mm to (84.9, 94.8), turned to 0 degrees
- moved R105 66.1 mm to (77.5, 109.0), turned to 90 degrees
- moved R106 63.3 mm to (80.0, 109.0), turned to 90 degrees
- moved R505 57.4 mm to (86.0, 78.4)
- moved R501 56.6 mm to (89.0, 81.2), turned to 90 degrees
- moved R605 55.9 mm to (118.9, 118.8)
- moved R601 54.4 mm to (118.9, 108.8)
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- renumbered D801 to D701, D701 to D801, D702 to D802, D703 to D803, J102 to J101, J103 to J102, J101 to J103, J801 to J701, J701 to J801, J702 to J802, J703 to J803, J704 to J804, J705 to J805, J706 to J806, J707 to J807, J708 to J808, JP202 to JP201, JP201 to JP202, JP503 to JP501, JP501 to JP503, K801 to K701, Q801 to Q701, R104 to R101, R105 to R102, R106 to R103, R107 to R104, R108 to R105, R109 to R106, R103 to R107, R101 to R108, R102 to R109, R121 to R114, R114 to R115, R115 to R116, R116 to R117, R117 to R118, R118 to R119, R119 to R120, R120 to R121, R203 to R201, R204 to R202, R205 to R203, R206 to R204, R202 to R205, R201 to R206, R305 to R302, R304 to R303, R302 to R304, R303 to R305, R403 to R402, R402 to R403, R604 to R602, R602 to R603, R605 to R604, R603 to R605, R801 to R701, R802 to R702, R804 to R704, R803 to R705, R805 to R706, R701 to R801, R702 to R802, R703 to R803, R704 to R804, R705 to R805, R706 to R806, R707 to R807, R708 to R808, SW701 to SW801
Connections:
- net /PiCoupler/READY renamed Net-(J701-Pin_29)
- J501 pad 1: /VCC_S1 -> /Power/VCC_CON1
- J502 pad 1: /VCC_S2 -> /Power/VCC_CON2
- J503 pad 1: /VCC_S3 -> /Power/VCC_CON3
- J504 pad 1: /VCC_S4 -> /Power/VCC_CON4
- Q501 pad 2: /VCC_S1 -> /Power/VCC_CON1
- Q502 pad 2: /VCC_S2 -> /Power/VCC_CON2
- Q503 pad 2: /VCC_S3 -> /Power/VCC_CON3
- Q504 pad 2: /VCC_S4 -> /Power/VCC_CON4
- R701 pad 1: /PiCoupler/POWERON -> /VCC_S8
- R804 pad 2: /CAMP -> Net-(R804-Pad2)
- R805 pad 2: /CAMP -> Net-(R804-Pad2)
- R806 pad 2: /CAMP -> Net-(R804-Pad2)
- R807 pad 2: /CAMP -> Net-(R804-Pad2)
- R808 pad 1: /CAMP -> Net-(R804-Pad2)
- U101 pad 34: unconnected-(U101-GPIO28_ADC2-Pad34) -> /CPU_READY
- U601 pad 8: /VCC_S1 -> /VCC_S5
Routing:
- net Net-(R804-Pad2): track 0.00 -> 180.1 mm
- net /SDA: track 19.4 -> 144.0 mm, vias 0 -> 1
- net /SCL: track 19.6 -> 141.5 mm, vias 0 -> 1
- net /UART_TX: track 0.00 -> 82.1 mm
- net /UART_RX: track 0.00 -> 77.0 mm
- net /GPS_PPS: track 0.00 -> 72.8 mm, vias 0 -> 2
- net Net-(U601-BUSY): track 0.00 -> 71.6 mm
- net /TTY_RX: track 0.00 -> 71.6 mm
- net /GPS_FIX: track 0.00 -> 68.4 mm, vias 0 -> 2
- net /TTY_TX: track 0.00 -> 67.8 mm
- net /Power/VPOW: track 0.00 -> 64.7 mm, vias 0 -> 4
- net Net-(U601-RST): track 0.00 -> 63.1 mm
- net /Power/VCC_CON4: track 0.00 -> 59.9 mm
- net /SW_VCC1: track 0.00 -> 59.3 mm, vias 0 -> 2
- net /Power/VCC_CON3: track 0.00 -> 55.6 mm, vias 0 -> 2
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- added copper zone on F.Cu, net GND
Other:
- board text added: "BSY RST DC CS CLK DIN GND VCC"
- board text added: "CH 1 2 3 4"
- board text added: "GND TX RX FIX PPS"
- board text added: "I²C"
- board text added: "ON/OFF"
- board text added: "SWDIO"
- board text added: "UART1 GPS"
- board text added: "eInk-Display"
- board text added: "override power-fets"
- board text removed: "J102=GPS U601=eInk"
- board text removed: "⏚ TX RX FIX PPS"

Commit message: finished first routing pass
Parts:
- removed J801, J802, J803, J804, J805, J806, J807, J808: Conn_01x14_Male, Connector_PinHeader_2.54mm:PinHeader_1x14_P2.54mm_Vertical
- moved R703 55.9 mm to (59.8, 144.3)
- moved R705 45.9 mm to (59.8, 147.7), turned to -90 degrees
- moved R509 42.8 mm to (85.0, 75.5), turned to -90 degrees
- moved R303 4.88 mm to (100.5, 89.2), turned to -90 degrees
- moved R302 4.85 mm to (100.6, 102.2), turned to -90 degrees
- moved R301 4.79 mm to (100.6, 107.0), turned to -90 degrees
- moved R305 4.74 mm to (100.6, 95.3), turned to 90 degrees
- moved R304 4.70 mm to (100.6, 98.7), turned to 90 degrees
- moved R809 0.40 mm to (75.1, 138.9)
Connections:
- K701 pad 11: +3.3V -> +BATT
Routing:
- net +3.3V: track 0.00 -> 281.2 mm, vias 0 -> 8
- net /LED1: track 0.00 -> 146.0 mm, vias 1 -> 2
- net GND: track 12.1 -> 152.3 mm, vias 10 -> 15
- net /VCC_S2: track 24.5 -> 160.8 mm, vias 4 -> 5
- net /LED2: track 0.00 -> 131.4 mm, vias 1 -> 2
- net /LED3: track 0.00 -> 124.3 mm, vias 1 -> 2
- net /VCC_S1: track 10.2 -> 125.7 mm
- net /VCC_S3: track 10.2 -> 104.0 mm
- net /VCC_S8: track 10.2 -> 73.2 mm, vias 4 -> 9
- net /VCC_S5: track 10.2 -> 64.2 mm, vias 4 -> 7
- net Net-(U101-GPIO26_ADC0): track 1.84 -> 48.7 mm, vias 0 -> 2
- net /SW_VCC4: track 35.1 -> 74.7 mm, vias 2 -> 1
- net Net-(J701-Pin_29): track 7.02 -> 43.8 mm, vias 1 -> 2
- net /SW_VCC3: track 43.0 -> 68.9 mm, vias 2 -> 1
- net /CPU_READY: track 0.00 -> 21.1 mm
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Other:
- board text added: "RUN"
