File: pouch2/hmi.kicad_sch (KiCad schematic)
At the start: 20 parts, among them J701 Conn_01x14_Male, J702 Conn_01x14_Male, J703 Conn_01x14_Male, J704 Conn_01x14_Male, J705 Conn_01x14_Male, J706 Conn_01x14_Male, J707 Conn_01x14_Male, J708 Conn_01x14_Male, SW701 SW_DIP_x08

Commit message: drawed a lot of things
Parts:
- added R809: 0, Resistor_SMD:R_0805_2012Metric, symbol Device:R
- renumbered D701 to D801, D702 to D802, D703 to D803, J701 to J801, J702 to J802, J703 to J803, J704 to J804, J705 to J805, J706 to J806, J707 to J807, J708 to J808, R701 to R801, R702 to R802, R703 to R803, R704 to R804, R705 to R805, R706 to R806, R707 to R807, R708 to R808, SW701 to SW801
Connections:
- net Campaign: now also R809.2; no longer R804.2, R805.2, R806.2, R807.2, R808.1
- new net: R804.2, R805.2, R806.2, R807.2, R808.1, R809.1
Changed lines of the file:
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@@
+	(wire
+		(pts
+			(xy 102.87 22.86) (xy 96.52 22.86)
+		)
+		(stroke
+			(width 0)
+			(type default)
+		)
+	)
 	(wire
 		(pts
@@
 	(wire
 		(pts
-			(xy 100.33 22.86) (xy 96.52 22.86)
+			(xy 115.57 22.86) (xy 110.49 22.86)
 		)
 		(stroke
@@
 	(hierarchical_label "Campaign"
 		(shape output)
-		(at 100.33 22.86 0)
+		(at 115.57 22.86 0)
 		(fields_autoplaced yes)
 		(effects
@@
 		(dnp no)
 		(fields_autoplaced yes)
-		(property "Reference" "#PWR0705"
+		(property "Reference" "#PWR0804"
 			(at 162.56 77.47 0)
 			(effects
@@
 			(project "pouch2"
 				(path "/278cfa6b-9496-4a22-b425-8abdb96793ef/dcbcf723-f7ed-4082-a41f-9f6fc76b941a"
-					(reference "#PWR0705")
+					(reference "#PWR0804")
 					(unit 1)
 				)
@@
 		(dnp no)
 		(fields_autoplaced yes)
-		(property "Reference" "#PWR0704"
+		(property "Reference" "#PWR0805"
 			(at 162.56 127 0)
 			(effects
@@
 			(project "pouch2"
 				(path "/278cfa6b-9496-4a22-b425-8abdb96793ef/dcbcf723-f7ed-4082-a41f-9f6fc76b941a"
-					(reference "#PWR0704")
+					(reference "#PWR0805")
 					(unit 1)
 				)
@@
 		(dnp no)
 		(fields_autoplaced yes)
-		(property "Reference" "R701"
+		(property "Reference" "R801"
 			(at 59.69 104.14 90)
 			(effects
@@
 			(project ""
 				(path "/278cfa6b-9496-4a22-b425-8abdb96793ef/dcbcf723-f7ed-4082-a41f-9f6fc76b941a"
-					(reference "R701")
+					(reference "R801")
 					(unit 1)
 				)
@@
 		(dnp no)
 		(fields_autoplaced yes)
-		(property "Reference" "#PWR0703"
+		(property "Reference" "#PWR0803"
 			(at 96.52 71.12 0)
 			(effects
@@
 			(project ""
 				(path "/278cfa6b-9496-4a22-b425-8abdb96793ef/dcbcf723-f7ed-4082-a41f-9f6fc76b941a"
-					(reference "#PWR0703")
+					(reference "#PWR0803")
 					(unit 1)
 				)
@@
 		(dnp no)
 		(fields_autoplaced yes)
-		(property "Reference" "R704"
+		(property "Reference" "R804"
 			(at 87.63 16.51 90)
 			(effects
@@
 			(project "pouch2"
 				(path "/278cfa6b-9496-4a22-b425-8abdb96793ef/dcbcf723-f7ed-4082-a41f-9f6fc76b941a"
-					(reference "R704")
+					(reference "R804")
 					(unit 1)
 				)
@@
 		(dnp no)
 		(fields_autoplaced yes)
-		(property "Reference" "R707"
+		(property "Reference" "R807"
 			(at 87.63 46.99 90)
 			(effects
@@
 			(project "pouch2"
 				(path "/278cfa6b-9496-4a22-b425-8abdb96793ef/dcbcf723-f7ed-4082-a41f-9f6fc76b941a"
-					(reference "R707")
+					(reference "R807")
 					(unit 1)
 				)
@@
 		(dnp no)
 		(fields_autoplaced yes)
-		(property "Reference" "D702"
+		(property "Reference" "D802"
 			(at 72.7075 115.57 0)
 			(effects
@@
 			(project "pouch2"
 				(path "/278cfa6b-9496-4a22-b425-8abdb96793ef/dcbcf723-f7ed-4082-a41f-9f6fc76b941a"
-					(reference "D702")
+					(reference "D802")
 					(unit 1)
 				)
@@
 		(dnp no)
 		(fields_autoplaced yes)
-		(property "Reference" "J705"
+		(property "Reference" "J805"
 			(at 220.345 87.63 0)
 			(effects
@@
 			(project "pouch2"
 				(path "/278cfa6b-9496-4a22-b425-8abdb96793ef/dcbcf723-f7ed-4082-a41f-9f6fc76b941a"
-					(reference "J705")
+					(reference "J805")
 					(unit 1)
 				)
@@
 		(dnp no)
 		(fields_autoplaced yes)
-		(property "Reference" "J702"
+		(property "Reference" "J802"
 			(at 173.355 87.63 0)
 			(effects
@@
 			(project "pouch2"
 				(path "/278cfa6b-9496-4a22-b425-8abdb96793ef/dcbcf723-f7ed-4082-a41f-9f6fc76b941a"
-					(reference "J702")
+					(reference "J802")
 					(unit 1)
 				)
@@
 		(dnp no)
 		(fields_autoplaced yes)
-		(property "Reference" "#PWR0701"
+		(property "Reference" "#PWR0801"
 			(at 31.75 41.91 0)
 			(effects
@@
 			(project ""
 				(path "/278cfa6b-9496-4a22-b425-8abdb96793ef/dcbcf723-f7ed-4082-a41f-9f6fc76b941a"
-					(reference "#PWR0701")
+					(reference "#PWR0801")
 					(unit 1)
 				)
@@
 		(dnp no)
 		(fields_autoplaced yes)
-		(property "Reference" "D703"
+		(property "Reference" "D803"
 			(at 72.7075 128.27 0)
 			(effects
@@
 			(project "pouch2"
 				(path "/278cfa6b-9496-4a22-b425-8abdb96793ef/dcbcf723-f7ed-4082-a41f-9f6fc76b941a"
-					(reference "D703")
+					(reference "D803")
 					(unit 1)
 				)
@@
 		(dnp no)
 		(fields_autoplaced yes)
-		(property "Reference" "R705"
+		(property "Reference" "R805"
 			(at 87.63 26.67 90)
 			(effects
@@
 			(project "pouch2"
 				(path "/278cfa6b-9496-4a22-b425-8abdb96793ef/dcbcf723-f7ed-4082-a41f-9f6fc76b941a"
-					(reference "R705")
+					(reference "R805")
 					(unit 1)
 				)
@@
 		(dnp no)
 		(fields_autoplaced yes)
-		(property "Reference" "R706"
+		(property "Reference" "R806"
 			(at 87.63 36.83 90)
 			(effects
@@
 			(project "pouch2"
 				(path "/278cfa6b-9496-4a22-b425-8abdb96793ef/dcbcf723-f7ed-4082-a41f-9f6fc76b941a"
-					(reference "R706")
+					(reference "R806")
+					(unit 1)
+				)
+			)
+		)
+	)
+	(symbol
+		(lib_id "Device:R")
+		(at 106.68 22.86 90)
+		(unit 1)
+		(exclude_from_sim no)
+		(in_bom yes)
+		(on_board yes)
+		(dnp no)
+		(fields_autoplaced yes)
+		(property "Reference" "R809"
+			(at 106.68 16.51 90)
+			(effects
+				(font
+					(size 1.27 1.27)
+				)
+			)
+		)
+		(property "Value" "0"
+			(at 106.68 19.05 90)
+			(effects
+				(font
+					(size 1.27 1.27)
+				)
+			)
+		)
+		(property "Footprint" "Resistor_SMD:R_0805_2012Metric"
+			(at 106.68 24.638 90)
+			(effects
+				(font
+					(size 1.27 1.27)
+				)
+				(hide yes)
+			)
+		)
+		(property "Datasheet" "~"
+			(at 106.68 22.86 0)
+			(effects
+				(font
+					(size 1.27 1.27)
+				)
+				(hide yes)
+			)
+		)
+		(property "Description" "Resistor"
+			(at 106.68 22.86 0)
+			(effects
+				(font
+					(size 1.27 1.27)
+				)
+				(hide yes)
+			)
+		)
+		(pin "1"
+		)
+		(pin "2"
+		)
+		(instances
+			(project ""
+				(path "/278cfa6b-9496-4a22-b425-8abdb96793ef/dcbcf723-f7ed-4082-a41f-9f6fc76b941a"
+					(reference "R809")
 					(unit 1)
 				)
@@
 		(dnp no)
 		(fields_autoplaced yes)
-		(property "Reference" "J707"
+		(property "Reference" "J807"
 			(at 253.365 87.63 0)
 			(effects
@@
 			(project "pouch2"
 				(path "/278cfa6b-9496-4a22-b425-8abdb96793ef/dcbcf723-f7ed-4082-a41f-9f6fc76b941a"
-					(reference "J707")
+					(reference "J807")
 					(unit 1)
 				)
@@
 		(dnp no)
 		(fields_autoplaced yes)
-		(property "Reference" "J701"
+		(property "Reference" "J801"
 			(at 158.115 87.63 0)
 			(effects
@@
 			(project ""
 				(path "/278cfa6b-9496-4a22-b425-8abdb96793ef/dcbcf723-f7ed-4082-a41f-9f6fc76b941a"
-					(reference "J701")
+					(reference "J801")
 					(unit 1)
 				)
@@
 		(dnp no)
 		(fields_autoplaced yes)
-		(property "Reference" "D701"
+		(property "Reference" "D801"
 			(at 72.7075 102.87 0)
 			(effects
@@
 			(project ""
 				(path "/278cfa6b-9496-4a22-b425-8abdb96793ef/dcbcf723-f7ed-4082-a41f-9f6fc76b941a"
-					(reference "D701")
+					(reference "D801")
 					(unit 1)
 				)
@@
 		(dnp no)
 		(fields_autoplaced yes)
-		(property "Reference" "R703"
+		(property "Reference" "R803"
 			(at 59.69 129.54 90)
 			(effects
@@
 			(project ""
 				(path "/278cfa6b-9496-4a22-b425-8abdb96793ef/dcbcf723-f7ed-4082-a41f-9f6fc76b941a"
-					(reference "R703")
+					(reference "R803")
 					(unit 1)
 				)
@@
 		(dnp no)
 		(fields_autoplaced yes)
-		(property "Reference" "SW701"
+		(property "Reference" "SW801"
 			(at 45.72 38.1 0)
 			(effects
@@
 			(project ""
 				(path "/278cfa6b-9496-4a22-b425-8abdb96793ef/dcbcf723-f7ed-4082-a41f-9f6fc76b941a"
-					(reference "SW701")
+					(reference "SW801")
 					(unit 1)
 				)
@@
 		(dnp no)
 		(fields_autoplaced yes)
-		(property "Reference" "R708"
+		(property "Reference" "R808"
 			(at 99.06 55.8799 0)
 			(effects
@@
 			(project ""
 				(path "/278cfa6b-9496-4a22-b425-8abdb96793ef/dcbcf723-f7ed-4082-a41f-9f6fc76b941a"
-					(reference "R708")
+					(reference "R808")
 					(unit 1)
 				)
@@
 		(dnp no)
 		(fields_autoplaced yes)
-		(property "Reference" "J708"
+		(property "Reference" "J808"
 			(at 268.605 87.63 0)
 			(effects
@@
 			(project "pouch2"
 				(path "/278cfa6b-9496-4a22-b425-8abdb96793ef/dcbcf723-f7ed-4082-a41f-9f6fc76b941a"
-					(reference "J708")
+					(reference "J808")
 					(unit 1)
 				)
@@
 		(dnp no)
 		(fields_autoplaced yes)
-		(property "Reference" "R702"
+		(property "Reference" "R802"
 			(at 59.69 116.84 90)
 			(effects
@@
 			(project ""
 				(path "/278cfa6b-9496-4a22-b425-8abdb96793ef/dcbcf723-f7ed-4082-a41f-9f6fc76b941a"
-					(reference "R702")
+					(reference "R802")
 					(unit 1)
 				)
@@
 		(dnp no)
 		(fields_autoplaced yes)
-		(property "Reference" "J703"
+		(property "Reference" "J803"
 			(at 191.135 87.63 0)
 			(effects
@@
 			(project "pouch2"
 				(path "/278cfa6b-9496-4a22-b425-8abdb96793ef/dcbcf723-f7ed-4082-a41f-9f6fc76b941a"
-					(reference "J703")
+					(reference "J803")
 					(unit 1)
 				)
@@
 		(dnp no)
 		(fields_autoplaced yes)
-		(property "Reference" "J706"
+		(property "Reference" "J806"
 			(at 235.585 87.63 0)
 			(effects
@@
 			(project "pouch2"
 				(path "/278cfa6b-9496-4a22-b425-8abdb96793ef/dcbcf723-f7ed-4082-a41f-9f6fc76b941a"
-					(reference "J706")
+					(reference "J806")
 					(unit 1)
 				)
@@
 		(dnp no)
 		(fields_autoplaced yes)
-		(property "Reference" "J704"
+		(property "Reference" "J804"
 			(at 206.375 87.63 0)
 			(effects
@@
 			(project "pouch2"
 				(path "/278cfa6b-9496-4a22-b425-8abdb96793ef/dcbcf723-f7ed-4082-a41f-9f6fc76b941a"
-					(reference "J704")
+					(reference "J804")
 					(unit 1)
 				)
@@
 		(dnp no)
 		(fields_autoplaced yes)
-		(property "Reference" "#PWR0702"
+		(property "Reference" "#PWR0802"
 			(at 81.28 148.59 0)
 			(effects
@@
 			(project ""
 				(path "/278cfa6b-9496-4a22-b425-8abdb96793ef/dcbcf723-f7ed-4082-a41f-9f6fc76b941a"
-					(reference "#PWR0702")
+					(reference "#PWR0802")
 					(unit 1)
 				)

Commit message: finished first routing pass
Parts:
- removed J801, J802, J803, J804, J805, J806, J807, J808: Conn_01x14_Male, Connector_PinHeader_2.54mm:PinHeader_1x14_P2.54mm_Vertical, symbol Connector:Conn_01x14_Male

Commit message: added VCC-battery measurement line
Parts:
- R801, R802, R803: LCSC (none) -> C17630; MPN_Eurocircuit (none) -> GPR0805330R
- R804: LCSC (none) -> C17840; MPN_Eurocircuit (none) -> GPR080582K
- R805: LCSC (none) -> C17713; MPN_Eurocircuit (none) -> GPR080547K
- R806: LCSC (none) -> C17560; MPN_Eurocircuit (none) -> GPR080522K
- R807, R808: LCSC (none) -> C17414; MPN_Eurocircuit (none) -> GPR080510K
- R809: LCSC (none) -> C17477; MPN_Eurocircuit (none) -> GPR08050R
Changed lines of the file:
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@@
+			)
+		)
+		(property "LCSC" "C17630"
+			(at 59.69 110.49 0)
+			(effects
+				(font
+					(size 1.27 1.27)
+				)
+				(hide yes)
+			)
+		)
+		(property "MPN_Eurocircuit" "GPR0805330R"
+			(at 59.69 110.49 0)
+			(effects
+				(font
+					(size 1.27 1.27)
+				)
+				(hide yes)
 			)
 		)
@@
 			)
 		)
+		(property "LCSC" "C17840"
+			(at 87.63 22.86 0)
+			(effects
+				(font
+					(size 1.27 1.27)
+				)
+				(hide yes)
+			)
+		)
+		(property "MPN_Eurocircuit" "GPR080582K"
+			(at 87.63 22.86 0)
+			(effects
+				(font
+					(size 1.27 1.27)
+				)
+				(hide yes)
+			)
+		)
 		(pin "1"
 		)
@@
 			)
 		)
+		(property "LCSC" "C17414"
+			(at 87.63 53.34 0)
+			(effects
+				(font
+					(size 1.27 1.27)
+				)
+				(hide yes)
+			)
+		)
+		(property "MPN_Eurocircuit" "GPR080510K"
+			(at 87.63 53.34 0)
+			(effects
+				(font
+					(size 1.27 1.27)
+				)
+				(hide yes)
+			)
+		)
 		(pin "1"
 		)
@@
 			)
 		)
+		(property "MPN_Eurocircuit" ""
+			(at 71.12 123.19 0)
+			(effects
+				(font
+					(size 1.27 1.27)
+				)
+				(hide yes)
+			)
+		)
 		(pin "2"
 		)
@@
 			)
 		)
+		(property "MPN_Eurocircuit" ""
+			(at 71.12 135.89 0)
+			(effects
+				(font
+					(size 1.27 1.27)
+				)
+				(hide yes)
+			)
+		)
 		(pin "2"
 		)
@@
 			)
 		)
+		(property "LCSC" "C17713"
+			(at 87.63 33.02 0)
+			(effects
+				(font
+					(size 1.27 1.27)
+				)
+				(hide yes)
+			)
+		)
+		(property "MPN_Eurocircuit" "GPR080547K"
+			(at 87.63 33.02 0)
+			(effects
+				(font
+					(size 1.27 1.27)
+				)
+				(hide yes)
+			)
+		)
 		(pin "1"
 		)
@@
 			)
 		)
+		(property "LCSC" "C17560"
+			(at 87.63 43.18 0)
+			(effects
+				(font
+					(size 1.27 1.27)
+				)
+				(hide yes)
+			)
+		)
+		(property "MPN_Eurocircuit" "GPR080522K"
+			(at 87.63 43.18 0)
+			(effects
+				(font
+					(size 1.27 1.27)
+				)
+				(hide yes)
+			)
+		)
 		(pin "1"
 		)
@@
 			)
 		)
+		(property "LCSC" "C17477"
+			(at 106.68 22.86 0)
+			(effects
+				(font
+					(size 1.27 1.27)
+				)
+				(hide yes)
+			)
+		)
+		(property "MPN_Eurocircuit" "GPR08050R"
+			(at 106.68 22.86 0)
+			(effects
+				(font
+					(size 1.27 1.27)
+				)
+				(hide yes)
+			)
+		)
 		(pin "1"
 		)
@@
 			)
 		)
+		(property "MPN_Eurocircuit" ""
+			(at 71.12 110.49 0)
+			(effects
+				(font
+					(size 1.27 1.27)
+				)
+				(hide yes)
+			)
+		)
 		(pin "2"
 		)
@@
 			)
 		)
+		(property "LCSC" "C17630"
+			(at 59.69 135.89 0)
+			(effects
+				(font
+					(size 1.27 1.27)
+				)
+				(hide yes)
+			)
+		)
+		(property "MPN_Eurocircuit" "GPR0805330R"
+			(at 59.69 135.89 0)
+			(effects
+				(font
+					(size 1.27 1.27)
+				)
+				(hide yes)
+			)
+		)
 		(pin "1"
 		)
@@
 			)
 		)
+		(property "MPN_Eurocircuit" ""
+			(at 45.72 55.88 0)
+			(effects
+				(font
+					(size 1.27 1.27)
+				)
+				(hide yes)
+			)
+		)
 		(pin "3"
 		)
@@
 			)
 		)
+		(property "LCSC" "C17414"
+			(at 96.52 57.15 0)
+			(effects
+				(font
+					(size 1.27 1.27)
+				)
+				(hide yes)
+			)
+		)
+		(property "MPN_Eurocircuit" "GPR080510K"
+			(at 96.52 57.15 0)
+			(effects
+				(font
+					(size 1.27 1.27)
+				)
+				(hide yes)
+			)
+		)
 		(pin "1"
 		)
@@
 			(at 59.69 123.19 0)
 			(effects
+				(font
+					(size 1.27 1.27)
+				)
+				(hide yes)
+			)
+		)
+		(property "LCSC" "C17630"
+			(at 59.69 123.19 0)
+			(effects
+				(font
+					(size 1.27 1.27)
+				)
+				(hide yes)
+			)
+		)
+		(property "MPN_Eurocircuit" "GPR0805330R"
+			(at 59.69 123.19 0)
+			(effects
