File: pouch2/hmi.kicad_sch (KiCad schematic)
At the start: 13 parts, among them SW801 SW_DIP_x08

Commit message: rev1
Parts:
- D801, D802, D803: OrderStatus (none) -> order
- R801, R802, R803, R804, R805, R806, R807, R808, R809: OrderStatus (none) -> assembly
- SW801: OrderStatus (none) -> manual
Changed lines of the file:
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@@
+	(wire
+		(pts
+			(xy 74.93 135.89) (xy 81.28 135.89)
+		)
+		(stroke
+			(width 0)
+			(type default)
+		)
+	)
 	(wire
 		(pts
@@
 	(wire
 		(pts
-			(xy 74.93 135.89) (xy 81.28 135.89)
+			(xy 53.34 53.34) (xy 83.82 53.34)
 		)
 		(stroke
@@
 	(wire
 		(pts
-			(xy 53.34 53.34) (xy 83.82 53.34)
+			(xy 91.44 33.02) (xy 96.52 33.02)
 		)
 		(stroke
@@
 	(wire
 		(pts
-			(xy 91.44 33.02) (xy 96.52 33.02)
+			(xy 96.52 60.96) (xy 96.52 64.77)
 		)
 		(stroke
@@
 	(wire
 		(pts
-			(xy 96.52 60.96) (xy 96.52 64.77)
+			(xy 63.5 110.49) (xy 67.31 110.49)
 		)
 		(stroke
@@
 	(wire
 		(pts
-			(xy 63.5 110.49) (xy 67.31 110.49)
-		)
-		(stroke
-			(width 0)
-			(type default)
-		)
-	)
-	(wire
-		(pts
-			(xy 81.28 135.89) (xy 81.28 142.24)
+			(xy 81.28 135.89) (xy 81.28 165.1)
 		)
 		(stroke
@@
 			)
 		)
+		(property "OrderStatus" "assembly"
+			(at 59.69 110.49 0)
+			(effects
+				(font
+					(size 1.27 1.27)
+				)
+				(hide yes)
+			)
+		)
 		(pin "2"
 		)
@@
 			)
 		)
+		(property "OrderStatus" "assembly"
+			(at 87.63 22.86 0)
+			(effects
+				(font
+					(size 1.27 1.27)
+				)
+				(hide yes)
+			)
+		)
 		(pin "1"
 		)
@@
 			)
 		)
+		(property "OrderStatus" "assembly"
+			(at 87.63 53.34 0)
+			(effects
+				(font
+					(size 1.27 1.27)
+				)
+				(hide yes)
+			)
+		)
 		(pin "1"
 		)
@@
 			)
 		)
+		(property "OrderStatus" "order"
+			(at 71.12 123.19 0)
+			(effects
+				(font
+					(size 1.27 1.27)
+				)
+				(hide yes)
+			)
+		)
 		(pin "2"
 		)
@@
 			)
 		)
+		(property "OrderStatus" "order"
+			(at 71.12 135.89 0)
+			(effects
+				(font
+					(size 1.27 1.27)
+				)
+				(hide yes)
+			)
+		)
 		(pin "2"
 		)
@@
 			)
 		)
+		(property "OrderStatus" "assembly"
+			(at 87.63 33.02 0)
+			(effects
+				(font
+					(size 1.27 1.27)
+				)
+				(hide yes)
+			)
+		)
 		(pin "1"
 		)
@@
 			)
 		)
+		(property "OrderStatus" "assembly"
+			(at 87.63 43.18 0)
+			(effects
+				(font
+					(size 1.27 1.27)
+				)
+				(hide yes)
+			)
+		)
 		(pin "1"
 		)
@@
 			)
 		)
+		(property "OrderStatus" "assembly"
+			(at 106.68 22.86 0)
+			(effects
+				(font
+					(size 1.27 1.27)
+				)
+				(hide yes)
+			)
+		)
 		(pin "1"
 		)
@@
 			)
 		)
+		(property "OrderStatus" "order"
+			(at 71.12 110.49 0)
+			(effects
+				(font
+					(size 1.27 1.27)
+				)
+				(hide yes)
+			)
+		)
 		(pin "2"
 		)
@@
 			)
 		)
+		(property "OrderStatus" "assembly"
+			(at 59.69 135.89 0)
+			(effects
+				(font
+					(size 1.27 1.27)
+				)
+				(hide yes)
+			)
+		)
 		(pin "1"
 		)
@@
 			)
 		)
+		(property "OrderStatus" "manual"
+			(at 45.72 55.88 0)
+			(effects
+				(font
+					(size 1.27 1.27)
+				)
+				(hide yes)
+			)
+		)
 		(pin "3"
 		)
@@
 			)
 		)
+		(property "OrderStatus" "assembly"
+			(at 96.52 57.15 0)
+			(effects
+				(font
+					(size 1.27 1.27)
+				)
+				(hide yes)
+			)
+		)
 		(pin "1"
 		)
@@
 			)
 		)
+		(property "OrderStatus" "assembly"
+			(at 59.69 123.19 0)
+			(effects
+				(font
+					(size 1.27 1.27)
+				)
+				(hide yes)
+			)
+		)
 		(pin "1"
 		)
@@
 	(symbol
 		(lib_id "power:GND")
-		(at 81.28 142.24 0)
+		(at 81.28 165.1 0)
 		(unit 1)
 		(exclude_from_sim no)
@@
 		(fields_autoplaced yes)
 		(property "Reference" "#PWR0802"
-			(at 81.28 148.59 0)
+			(at 81.28 171.45 0)
 			(effects
 				(font
@@
 		)
 		(property "Value" "GND"
-			(at 81.28 147.32 0)
+			(at 81.28 170.18 0)
 			(effects
 				(font
@@
 		)
 		(property "Footprint" ""
-			(at 81.28 142.24 0)
+			(at 81.28 165.1 0)
 			(effects
 				(font
@@
 		)
 		(property "Datasheet" ""
-			(at 81.28 142.24 0)
+			(at 81.28 165.1 0)
 			(effects
 				(font
@@
 		)
 		(property "Description" "Power symbol creates a global label with name \"GND\" , ground"
-			(at 81.28 142.24 0)
-			(effects
-				(font
+			(at 81.28 165.1 0)
+			(effects
+				(font
