File: pouch2/accel_gyro.kicad_sch (KiCad schematic)
At the start: 15 parts, among them U201 BME688, U202 BME280

Commit message: drawed a lot of things
Parts:
- renumbered JP202 to JP201, JP201 to JP202, R203 to R201, R204 to R202, R205 to R203, R206 to R204, R202 to R205, R201 to R206
Changed lines of the file:
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@@
 		(dnp no)
 		(fields_autoplaced yes)
-		(property "Reference" "R203"
+		(property "Reference" "R201"
 			(at 71.12 140.97 90)
 			(effects
@@
 			(project "pouch2"
 				(path "/278cfa6b-9496-4a22-b425-8abdb96793ef/245dc3ad-3701-4382-b188-f6e1df98764a"
-					(reference "R203")
+					(reference "R201")
 					(unit 1)
 				)
@@
 		(dnp no)
 		(fields_autoplaced yes)
-		(property "Reference" "JP201"
+		(property "Reference" "JP202"
 			(at 116.84 140.9699 90)
 			(effects
@@
 			(project "pouch2"
 				(path "/278cfa6b-9496-4a22-b425-8abdb96793ef/245dc3ad-3701-4382-b188-f6e1df98764a"
-					(reference "JP201")
+					(reference "JP202")
 					(unit 1)
 				)
@@
 		(dnp no)
 		(fields_autoplaced yes)
-		(property "Reference" "#PWR0204"
+		(property "Reference" "#PWR0206"
 			(at 114.3 143.51 0)
 			(effects
@@
 			(project "pouch2"
 				(path "/278cfa6b-9496-4a22-b425-8abdb96793ef/245dc3ad-3701-4382-b188-f6e1df98764a"
-					(reference "#PWR0204")
+					(reference "#PWR0206")
 					(unit 1)
 				)
@@
 		(dnp no)
 		(fields_autoplaced yes)
-		(property "Reference" "R204"
+		(property "Reference" "R202"
 			(at 71.12 158.75 90)
 			(effects
@@
 			(project "pouch2"
 				(path "/278cfa6b-9496-4a22-b425-8abdb96793ef/245dc3ad-3701-4382-b188-f6e1df98764a"
-					(reference "R204")
+					(reference "R202")
 					(unit 1)
 				)
@@
 		(dnp no)
 		(fields_autoplaced yes)
-		(property "Reference" "JP202"
+		(property "Reference" "JP201"
 			(at 106.68 48.2599 90)
 			(effects
@@
 			(project "pouch2"
 				(path "/278cfa6b-9496-4a22-b425-8abdb96793ef/245dc3ad-3701-4382-b188-f6e1df98764a"
-					(reference "JP202")
+					(reference "JP201")
 					(unit 1)
 				)
@@
 		(dnp no)
 		(fields_autoplaced yes)
-		(property "Reference" "#PWR0203"
+		(property "Reference" "#PWR0205"
 			(at 114.3 127 0)
 			(effects
@@
 			(project "pouch2"
 				(path "/278cfa6b-9496-4a22-b425-8abdb96793ef/245dc3ad-3701-4382-b188-f6e1df98764a"
-					(reference "#PWR0203")
+					(reference "#PWR0205")
 					(unit 1)
 				)
@@
 		(on_board yes)
 		(dnp no)
-		(property "Reference" "R206"
+		(property "Reference" "R204"
 			(at 73.914 64.008 90)
 			(effects
@@
 			(project "pouch2"
 				(path "/278cfa6b-9496-4a22-b425-8abdb96793ef/245dc3ad-3701-4382-b188-f6e1df98764a"
-					(reference "R206")
+					(reference "R204")
 					(unit 1)
 				)
@@
 		(dnp no)
 		(fields_autoplaced yes)
-		(property "Reference" "R202"
+		(property "Reference" "R205"
 			(at 93.98 43.18 90)
 			(effects
@@
 			(project "pouch2"
 				(path "/278cfa6b-9496-4a22-b425-8abdb96793ef/245dc3ad-3701-4382-b188-f6e1df98764a"
-					(reference "R202")
+					(reference "R205")
 					(unit 1)
 				)
@@
 		(on_board yes)
 		(dnp no)
-		(property "Reference" "R205"
+		(property "Reference" "R203"
 			(at 73.66 50.8 90)
 			(effects
@@
 			(project "pouch2"
 				(path "/278cfa6b-9496-4a22-b425-8abdb96793ef/245dc3ad-3701-4382-b188-f6e1df98764a"
-					(reference "R205")
+					(reference "R203")
 					(unit 1)
 				)
@@
 		(dnp no)
 		(fields_autoplaced yes)
-		(property "Reference" "R201"
+		(property "Reference" "R206"
 			(at 99.06 135.89 90)
 			(effects
@@
 			(project "pouch2"
 				(path "/278cfa6b-9496-4a22-b425-8abdb96793ef/245dc3ad-3701-4382-b188-f6e1df98764a"
-					(reference "R201")
+					(reference "R206")
 					(unit 1)
 				)
@@
 		(dnp no)
 		(fields_autoplaced yes)
-		(property "Reference" "#PWR0205"
+		(property "Reference" "#PWR0203"
 			(at 104.14 38.1 0)
 			(effects
@@
 			(project "pouch2"
 				(path "/278cfa6b-9496-4a22-b425-8abdb96793ef/245dc3ad-3701-4382-b188-f6e1df98764a"
-					(reference "#PWR0205")
+					(reference "#PWR0203")
 					(unit 1)
 				)
@@
 		(dnp no)
 		(fields_autoplaced yes)
-		(property "Reference" "#PWR0206"
+		(property "Reference" "#PWR0204"
 			(at 104.14 50.8 0)
 			(effects
@@
 			(project "pouch2"
 				(path "/278cfa6b-9496-4a22-b425-8abdb96793ef/245dc3ad-3701-4382-b188-f6e1df98764a"
-					(reference "#PWR0206")
-					(unit 1)
-				)
+					(reference "#PWR0204")
+					(unit 1)
+				)

Commit message: added VCC-battery measurement line
Parts:
- R201, R202, R203, R204, R207, R208: LCSC (none) -> C17477; MPN_Eurocircuit (none) -> GPR08050R
- R205, R206, R209: LCSC (none) -> C17560; MPN_Eurocircuit (none) -> GPR080522K
Changed lines of the file:
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@@
+			)
+		)
+		(property "LCSC" "C17477"
+			(at 71.12 147.32 0)
+			(effects
+				(font
+					(size 1.27 1.27)
+				)
+				(hide yes)
+			)
+		)
+		(property "MPN_Eurocircuit" "GPR08050R"
+			(at 71.12 147.32 0)
+			(effects
+				(font
+					(size 1.27 1.27)
+				)
+				(hide yes)
 			)
 		)
@@
 			)
 		)
+		(property "MPN_Eurocircuit" ""
+			(at 114.3 142.24 0)
+			(effects
+				(font
+					(size 1.27 1.27)
+				)
+				(hide yes)
+			)
+		)
 		(pin "1"
 		)
@@
 			)
 		)
+		(property "MPN_Eurocircuit" ""
+			(at 194.31 78.74 0)
+			(effects
+				(font
+					(size 1.27 1.27)
+				)
+				(hide yes)
+			)
+		)
 		(pin "1"
 		)
@@
 			)
 		)
+		(property "LCSC" "C17477"
+			(at 194.31 62.23 0)
+			(effects
+				(font
+					(size 1.27 1.27)
+				)
+				(hide yes)
+			)
+		)
+		(property "MPN_Eurocircuit" "GPR08050R"
+			(at 194.31 62.23 0)
+			(effects
+				(font
+					(size 1.27 1.27)
+				)
+				(hide yes)
+			)
+		)
 		(pin "2"
 		)
@@
 			)
 		)
+		(property "MPN_Eurocircuit" ""
+			(at 41.91 57.15 0)
+			(effects
+				(font
+					(size 1.27 1.27)
+				)
+				(hide yes)
+			)
+		)
 		(pin "3"
 		)
@@
 			)
 		)
+		(property "LCSC" "C17477"
+			(at 71.12 152.4 0)
+			(effects
+				(font
+					(size 1.27 1.27)
+				)
+				(hide yes)
+			)
+		)
+		(property "MPN_Eurocircuit" "GPR08050R"
+			(at 71.12 152.4 0)
+			(effects
+				(font
+					(size 1.27 1.27)
+				)
+				(hide yes)
+			)
+		)
 		(pin "2"
 		)
@@
 			)
 		)
+		(property "MPN_Eurocircuit" ""
+			(at 104.14 49.53 0)
+			(effects
+				(font
+					(size 1.27 1.27)
+				)
+				(hide yes)
+			)
+		)
 		(pin "1"
 		)
@@
 			)
 		)
+		(property "MPN_Eurocircuit" ""
+			(at 224.79 59.69 0)
+			(effects
+				(font
+					(size 1.27 1.27)
+				)
+				(hide yes)
+			)
+		)
 		(pin "3"
 		)
@@
 			)
 		)
+		(property "LCSC" "C17477"
+			(at 73.66 59.69 0)
+			(effects
+				(font
+					(size 1.27 1.27)
+				)
+				(hide yes)
+			)
+		)
+		(property "MPN_Eurocircuit" "GPR08050R"
+			(at 73.66 59.69 0)
+			(effects
+				(font
+					(size 1.27 1.27)
+				)
+				(hide yes)
+			)
+		)
 		(pin "2"
 		)
@@
 			)
 		)
+		(property "LCSC" "C17560"
+			(at 93.98 49.53 0)
+			(effects
+				(font
+					(size 1.27 1.27)
+				)
+				(hide yes)
+			)
+		)
+		(property "MPN_Eurocircuit" "GPR080522K"
+			(at 93.98 49.53 0)
+			(effects
+				(font
+					(size 1.27 1.27)
+				)
+				(hide yes)
+			)
+		)
 		(pin "1"
 		)
@@
 			)
 		)
+		(property "LCSC" "C17477"
+			(at 73.66 54.61 0)
+			(effects
+				(font
+					(size 1.27 1.27)
+				)
+				(hide yes)
+			)
+		)
+		(property "MPN_Eurocircuit" "GPR08050R"
+			(at 73.66 54.61 0)
+			(effects
+				(font
+					(size 1.27 1.27)
+				)
+				(hide yes)
+			)
+		)
 		(pin "2"
 		)
@@
 			)
 		)
+		(property "LCSC" "C17477"
+			(at 194.31 52.07 0)
+			(effects
+				(font
+					(size 1.27 1.27)
+				)
+				(hide yes)
+			)
+		)
+		(property "MPN_Eurocircuit" "GPR08050R"
+			(at 194.31 52.07 0)
+			(effects
+				(font
+					(size 1.27 1.27)
+				)
+				(hide yes)
+			)
+		)
 		(pin "2"
 		)
@@
 			)
 		)
+		(property "LCSC" "C17560"
+			(at 99.06 142.24 0)
+			(effects
+				(font
+					(size 1.27 1.27)
+				)
+				(hide yes)
+			)
+		)
+		(property "MPN_Eurocircuit" "GPR080522K"
+			(at 99.06 142.24 0)
+			(effects
+				(font
+					(size 1.27 1.27)
+				)
+				(hide yes)
+			)
+		)
 		(pin "1"
 		)
@@
 			)
 		)
+		(property "MPN_Eurocircuit" ""
+			(at 41.91 149.86 0)
+			(effects
+				(font
+					(size 1.27 1.27)
+				)
+				(hide yes)
+			)
+		)
 		(pin "5"
 		)
@@
 			(at 203.2 74.93 0)
 			(effects
+				(font
+					(size 1.27 1.27)
+				)
+				(hide yes)
+			)
+		)
+		(property "LCSC" "C17560"
+			(at 203.2 74.93 0)
+			(effects
+				(font
+					(size 1.27 1.27)
+				)
+				(hide yes)
+			)
+		)
+		(property "MPN_Eurocircuit" "GPR080522K"
+			(at 203.2 74.93 0)
+			(effects

Commit message: rev1
Parts:
- JP201, JP202, JP203: OrderStatus (none) -> dnp
- R201, R202, R203, R204, R205, R206, R207, R208, R209: OrderStatus (none) -> assembly
- U201, U202, XX201: OrderStatus (none) -> manual
Changed lines of the file:
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@@
+			)
+		)
+		(property "OrderStatus" "assembly"
+			(at 71.12 147.32 0)
+			(effects
+				(font
+					(size 1.27 1.27)
+				)
+				(hide yes)
 			)
 		)
@@
 			)
 		)
+		(property "OrderStatus" "dnp"
+			(at 114.3 142.24 0)
+			(effects
+				(font
+					(size 1.27 1.27)
+				)
+				(hide yes)
+			)
+		)
 		(pin "1"
 		)
@@
 			)
 		)
+		(property "OrderStatus" "dnp"
+			(at 194.31 78.74 0)
+			(effects
+				(font
+					(size 1.27 1.27)
+				)
+				(hide yes)
+			)
+		)
 		(pin "1"
 		)
@@
 			)
 		)
+		(property "OrderStatus" "assembly"
+			(at 194.31 62.23 0)
+			(effects
+				(font
+					(size 1.27 1.27)
+				)
+				(hide yes)
+			)
+		)
 		(pin "2"
 		)
@@
 			)
 		)
+		(property "OrderStatus" "manual"
+			(at 41.91 57.15 0)
+			(effects
+				(font
+					(size 1.27 1.27)
+				)
+				(hide yes)
+			)
+		)
 		(pin "3"
 		)
@@
 			)
 		)
+		(property "OrderStatus" "assembly"
+			(at 71.12 152.4 0)
+			(effects
+				(font
+					(size 1.27 1.27)
+				)
+				(hide yes)
+			)
+		)
 		(pin "2"
 		)
@@
 			)
 		)
+		(property "OrderStatus" "dnp"
+			(at 104.14 49.53 0)
+			(effects
+				(font
+					(size 1.27 1.27)
+				)
+				(hide yes)
+			)
+		)
 		(pin "1"
 		)
@@
 			)
 		)
+		(property "OrderStatus" "manual"
+			(at 224.79 59.69 0)
+			(effects
+				(font
+					(size 1.27 1.27)
+				)
+				(hide yes)
+			)
+		)
 		(pin "3"
 		)
@@
 			)
 		)
+		(property "OrderStatus" "assembly"
+			(at 73.66 59.69 0)
+			(effects
+				(font
+					(size 1.27 1.27)
+				)
+				(hide yes)
+			)
+		)
 		(pin "2"
 		)
@@
 			)
 		)
+		(property "OrderStatus" "assembly"
+			(at 93.98 49.53 0)
+			(effects
+				(font
+					(size 1.27 1.27)
+				)
+				(hide yes)
+			)
+		)
 		(pin "1"
 		)
@@
 			)
 		)
+		(property "OrderStatus" "assembly"
+			(at 73.66 54.61 0)
+			(effects
+				(font
+					(size 1.27 1.27)
+				)
+				(hide yes)
+			)
+		)
 		(pin "2"
 		)
@@
 			)
 		)
+		(property "OrderStatus" "assembly"
+			(at 194.31 52.07 0)
+			(effects
+				(font
+					(size 1.27 1.27)
+				)
+				(hide yes)
+			)
+		)
 		(pin "2"
 		)
@@
 			)
 		)
+		(property "OrderStatus" "assembly"
+			(at 99.06 142.24 0)
+			(effects
+				(font
+					(size 1.27 1.27)
+				)
+				(hide yes)
+			)
+		)
 		(pin "1"
 		)
@@
 			)
 		)
+		(property "OrderStatus" "manual"
+			(at 41.91 149.86 0)
+			(effects
+				(font
+					(size 1.27 1.27)
+				)
+				(hide yes)
+			)
+		)
 		(pin "5"
 		)
@@
 			(at 203.2 74.93 0)
 			(effects
+				(font
+					(size 1.27 1.27)
+				)
+				(hide yes)
+			)
+		)
+		(property "OrderStatus" "assembly"
+			(at 203.2 74.93 0)
+			(effects
