File: pouch2/eink_display.kicad_sch (KiCad schematic)
At the start: 1 part

Commit message: started PCB design
Parts:
- U601: renamed from U6; footprint (none) -> Connector_PinHeader_2.54mm:PinHeader_1x08_P2.54mm_Vertical
Changed lines of the file:
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@@
 		(dnp no)
 		(fields_autoplaced yes)
-		(property "Reference" "U6"
+		(property "Reference" "U601"
 			(at 130.81 79.3749 0)
 			(effects
@@
 			)
 		)
-		(property "Footprint" ""
+		(property "Footprint" "Connector_PinHeader_2.54mm:PinHeader_1x08_P2.54mm_Vertical"
 			(at 138.43 90.17 0)
 			(effects
@@
 			(project ""
 				(path "/278cfa6b-9496-4a22-b425-8abdb96793ef/b8350d3f-b373-4dd1-a1a4-91efa3226b27"
-					(reference "U6")
+					(reference "U601")
 					(unit 1)
 				)
@@
 		(dnp no)
 		(fields_autoplaced yes)
-		(property "Reference" "#PWR023"
+		(property "Reference" "#PWR0601"
 			(at 137.16 106.68 0)
 			(effects
@@
 			(project ""
 				(path "/278cfa6b-9496-4a22-b425-8abdb96793ef/b8350d3f-b373-4dd1-a1a4-91efa3226b27"
-					(reference "#PWR023")
+					(reference "#PWR0601")
 					(unit 1)
 				)

Commit message: started routing
Parts:
- added R601, R602, R603, R604, R605, R606: 0, Resistor_SMD:R_0805_2012Metric, symbol Device:R
Connections:
- net BUSY: now also R601.2; no longer U601.1 (BUSY)
- net CLK: now also R605.1; no longer U601.5 (CLK)
- net CS: now also R604.1; no longer U601.4 (CS)
- net DC: now also R603.2; no longer U601.3 (DC)
- net MOSI: now also R606.2; no longer U601.6 (DIN)
- net RST: now also R602.1; no longer U601.2 (RST)
- new net: R605.2, U601.5 (CLK)
- new net: R602.2, U601.2 (RST)
- new net: R601.1, U601.1 (BUSY)
- new net: R603.1, U601.3 (DC)
- new net: R604.2, U601.4 (CS)
- new net: R606.1, U601.6 (DIN)

Commit message: drawed a lot of things
Parts:
- renumbered R604 to R602, R602 to R603, R605 to R604, R603 to R605
Changed lines of the file:
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@@
 		(on_board yes)
 		(dnp no)
-		(property "Reference" "R605"
+		(property "Reference" "R604"
 			(at 164.084 82.55 90)
 			(effects
@@
 			(project ""
 				(path "/278cfa6b-9496-4a22-b425-8abdb96793ef/b8350d3f-b373-4dd1-a1a4-91efa3226b27"
-					(reference "R605")
+					(reference "R604")
 					(unit 1)
 				)
@@
 		(on_board yes)
 		(dnp no)
-		(property "Reference" "R602"
+		(property "Reference" "R603"
 			(at 164.084 72.39 90)
 			(effects
@@
 			(project ""
 				(path "/278cfa6b-9496-4a22-b425-8abdb96793ef/b8350d3f-b373-4dd1-a1a4-91efa3226b27"
-					(reference "R602")
+					(reference "R603")
 					(unit 1)
 				)
@@
 		(on_board yes)
 		(dnp no)
-		(property "Reference" "R604"
+		(property "Reference" "R602"
 			(at 156.464 80.01 90)
 			(effects
@@
 			(project ""
 				(path "/278cfa6b-9496-4a22-b425-8abdb96793ef/b8350d3f-b373-4dd1-a1a4-91efa3226b27"
-					(reference "R604")
+					(reference "R602")
 					(unit 1)
 				)
@@
 		(on_board yes)
 		(dnp no)
-		(property "Reference" "R603"
+		(property "Reference" "R605"
 			(at 171.45 74.93 90)
 			(effects
@@
 			(project ""
 				(path "/278cfa6b-9496-4a22-b425-8abdb96793ef/b8350d3f-b373-4dd1-a1a4-91efa3226b27"
-					(reference "R603")
-					(unit 1)
-				)
+					(reference "R605")
+					(unit 1)
+				)

Commit message: added VCC-battery measurement line
Parts:
- R601, R602, R603, R604, R605, R606: LCSC (none) -> C17477; MPN_Eurocircuit (none) -> GPR08050R
Changed lines of the file:
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@@
+			)
+		)
+		(property "LCSC" "C17477"
+			(at 163.83 85.09 0)
+			(effects
+				(font
+					(size 1.27 1.27)
+				)
+				(hide yes)
+			)
+		)
+		(property "MPN_Eurocircuit" "GPR08050R"
+			(at 163.83 85.09 0)
+			(effects
+				(font
+					(size 1.27 1.27)
+				)
+				(hide yes)
 			)
 		)
@@
 			)
 		)
+		(property "LCSC" "C17477"
+			(at 163.83 74.93 0)
+			(effects
+				(font
+					(size 1.27 1.27)
+				)
+				(hide yes)
+			)
+		)
+		(property "MPN_Eurocircuit" "GPR08050R"
+			(at 163.83 74.93 0)
+			(effects
+				(font
+					(size 1.27 1.27)
+				)
+				(hide yes)
+			)
+		)
 		(pin "1"
 		)
@@
 		)
 		(property "Description" "Resistor"
+			(at 156.21 72.39 0)
+			(effects
+				(font
+					(size 1.27 1.27)
+				)
+				(hide yes)
+			)
+		)
+		(property "LCSC" "C17477"
+			(at 156.21 72.39 0)
+			(effects
+				(font
+					(size 1.27 1.27)
+				)
+				(hide yes)
+			)
+		)
+		(property "MPN_Eurocircuit" "GPR08050R"
 			(at 156.21 72.39 0)
 			(effects
@@
 			)
 		)
+		(property "MPN_Eurocircuit" ""
+			(at 138.43 90.17 0)
+			(effects
+				(font
+					(size 1.27 1.27)
+				)
+				(hide yes)
+			)
+		)
 		(pin "7"
 		)
@@
 			)
 		)
+		(property "LCSC" "C17477"
+			(at 171.45 87.63 0)
+			(effects
+				(font
+					(size 1.27 1.27)
+				)
+				(hide yes)
+			)
+		)
+		(property "MPN_Eurocircuit" "GPR08050R"
+			(at 171.45 87.63 0)
+			(effects
+				(font
+					(size 1.27 1.27)
+				)
+				(hide yes)
+			)
+		)
 		(pin "1"
 		)
@@
 			)
 		)
+		(property "LCSC" "C17477"
+			(at 156.21 82.55 0)
+			(effects
+				(font
+					(size 1.27 1.27)
+				)
+				(hide yes)
+			)
+		)
+		(property "MPN_Eurocircuit" "GPR08050R"
+			(at 156.21 82.55 0)
+			(effects
+				(font
+					(size 1.27 1.27)
+				)
+				(hide yes)
+			)
+		)
 		(pin "2"
 		)
@@
 			(at 171.45 77.47 0)
 			(effects
+				(font
+					(size 1.27 1.27)
+				)
+				(hide yes)
+			)
+		)
+		(property "LCSC" "C17477"
+			(at 171.45 77.47 0)
+			(effects
+				(font
+					(size 1.27 1.27)
+				)
+				(hide yes)
+			)
+		)
+		(property "MPN_Eurocircuit" "GPR08050R"
+			(at 171.45 77.47 0)
+			(effects

Commit message: rev1
Parts:
- R601, R602, R603, R604, R605, R606: OrderStatus (none) -> assembly
- U601: OrderStatus (none) -> manual
Changed lines of the file:
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@@
+			)
+		)
+		(property "OrderStatus" "assembly"
+			(at 163.83 85.09 0)
+			(effects
+				(font
+					(size 1.27 1.27)
+				)
+				(hide yes)
 			)
 		)
@@
 			)
 		)
+		(property "OrderStatus" "assembly"
+			(at 163.83 74.93 0)
+			(effects
+				(font
+					(size 1.27 1.27)
+				)
+				(hide yes)
+			)
+		)
 		(pin "1"
 		)
@@
 		)
 		(property "MPN_Eurocircuit" "GPR08050R"
+			(at 156.21 72.39 0)
+			(effects
+				(font
+					(size 1.27 1.27)
+				)
+				(hide yes)
+			)
+		)
+		(property "OrderStatus" "assembly"
 			(at 156.21 72.39 0)
 			(effects
@@
 			)
 		)
+		(property "OrderStatus" "manual"
+			(at 138.43 90.17 0)
+			(effects
+				(font
+					(size 1.27 1.27)
+				)
+				(hide yes)
+			)
+		)
 		(pin "7"
 		)
@@
 			)
 		)
+		(property "OrderStatus" "assembly"
+			(at 171.45 87.63 0)
+			(effects
+				(font
+					(size 1.27 1.27)
+				)
+				(hide yes)
+			)
+		)
 		(pin "1"
 		)
@@
 			)
 		)
+		(property "OrderStatus" "assembly"
+			(at 156.21 82.55 0)
+			(effects
+				(font
+					(size 1.27 1.27)
+				)
+				(hide yes)
+			)
+		)
 		(pin "2"
 		)
@@
 			(at 171.45 77.47 0)
 			(effects
+				(font
+					(size 1.27 1.27)
+				)
+				(hide yes)
+			)
+		)
+		(property "OrderStatus" "assembly"
+			(at 171.45 77.47 0)
+			(effects
