File: pouch2/gps.kicad_sch (KiCad schematic)
At the start: 9 parts, among them U302 L86-M33

Commit message: rev1
Parts:
- R301, R302, R303, R304, R305: OrderStatus (none) -> assembly
- TP301, TP302: OrderStatus (none) -> dnp
- U301, U302: OrderStatus (none) -> manual
Changed lines of the file:
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@@
+			)
+		)
+		(property "OrderStatus" "assembly"
+			(at 190.5 74.93 0)
+			(effects
+				(font
+					(size 1.27 1.27)
+				)
+				(hide yes)
 			)
 		)
@@
 			)
 		)
+		(property "OrderStatus" "assembly"
+			(at 144.78 46.99 0)
+			(effects
+				(font
+					(size 1.27 1.27)
+				)
+				(hide yes)
+			)
+		)
 		(pin "2"
 		)
@@
 			)
 		)
+		(property "OrderStatus" "dnp"
+			(at 73.66 58.42 0)
+			(effects
+				(font
+					(size 1.27 1.27)
+				)
+				(hide yes)
+			)
+		)
 		(pin "1"
 		)
@@
 		)
 		(property "MPN_Eurocircuit" "GPR08050R"
+			(at 190.5 68.58 0)
+			(effects
+				(font
+					(size 1.27 1.27)
+				)
+				(hide yes)
+			)
+		)
+		(property "OrderStatus" "assembly"
 			(at 190.5 68.58 0)
 			(effects
@@
 			)
 		)
+		(property "OrderStatus" "dnp"
+			(at 73.66 68.58 0)
+			(effects
+				(font
+					(size 1.27 1.27)
+				)
+				(hide yes)
+			)
+		)
 		(pin "1"
 		)
@@
 		)
 		(property "MPN_Eurocircuit" "GPR08050R"
+			(at 190.5 58.42 0)
+			(effects
+				(font
+					(size 1.27 1.27)
+				)
+				(hide yes)
+			)
+		)
+		(property "OrderStatus" "assembly"
 			(at 190.5 58.42 0)
 			(effects
@@
 			)
 		)
+		(property "OrderStatus" "manual"
+			(at 158.75 83.82 0)
+			(effects
+				(font
+					(size 1.27 1.27)
+				)
+				(hide yes)
+			)
+		)
 		(pin "8"
 		)
@@
 			)
 		)
+		(property "OrderStatus" "manual"
+			(at 95.25 60.96 0)
+			(effects
+				(font
+					(size 1.27 1.27)
+				)
+				(hide yes)
+			)
+		)
 		(pin "6"
 		)
@@
 			(at 190.5 85.09 0)
 			(effects
+				(font
+					(size 1.27 1.27)
+				)
+				(hide yes)
+			)
+		)
+		(property "OrderStatus" "assembly"
+			(at 190.5 85.09 0)
+			(effects
