File: pouch2/pi_zero.kicad_sch (KiCad schematic)
At the start: 9 parts, among them J16 Conn_02x20_Odd_Even, K1 AZ9371-1A-5DE, Q5 MMBT3906

Commit message: started PCB design
Parts:
- J801: renamed from J16; value Conn_02x20_Odd_Even -> PiZero; footprint Connector_PinHeader_1.27mm:PinHeader_2x20_P1.27mm_Horizontal -> Module:Raspberry_Pi_Zero_Socketed_THT_FaceDown_MountingHoles; symbol Connector_Generic:Conn_02x20_Odd_Even -> SensorBoards:PiZero
- R801: renamed from R50; footprint Resistor_SMD:R_0815_2038Metric -> Resistor_SMD:R_0805_2012Metric
- R802: renamed from R51; footprint Resistor_SMD:R_0815_2038Metric -> Resistor_SMD:R_0805_2012Metric
- R803: renamed from R54; footprint Resistor_SMD:R_0815_2038Metric -> Resistor_SMD:R_0805_2012Metric
- R804: renamed from R53; footprint Resistor_SMD:R_0815_2038Metric -> Resistor_SMD:R_0805_2012Metric
- R805: renamed from R52; footprint Resistor_SMD:R_0815_2038Metric -> Resistor_SMD:R_0805_2012Metric
- renumbered D4 to D801, K1 to K801, Q5 to Q801
Changed lines of the file:
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@@
 		(dnp no)
 		(fields_autoplaced yes)
-		(property "Reference" "R51"
+		(property "Reference" "R802"
 			(at 78.74 57.1499 0)
 			(effects
@@
 			)
 		)
-		(property "Footprint" "Resistor_SMD:R_0815_2038Metric"
+		(property "Footprint" "Resistor_SMD:R_0805_2012Metric"
 			(at 77.978 58.42 90)
 			(effects
@@
 			(project ""
 				(path "/278cfa6b-9496-4a22-b425-8abdb96793ef/1f6da6ca-ffaf-4729-a842-c849ecc1a6dc"
-					(reference "R51")
+					(reference "R802")
 					(unit 1)
 				)
@@
 		(dnp no)
 		(fields_autoplaced yes)
-		(property "Reference" "R54"
+		(property "Reference" "R803"
 			(at 156.21 83.8199 0)
 			(effects
@@
 			)
 		)
-		(property "Footprint" "Resistor_SMD:R_0815_2038Metric"
+		(property "Footprint" "Resistor_SMD:R_0805_2012Metric"
 			(at 151.892 85.09 90)
 			(effects
@@
 			(project ""
 				(path "/278cfa6b-9496-4a22-b425-8abdb96793ef/1f6da6ca-ffaf-4729-a842-c849ecc1a6dc"
-					(reference "R54")
-					(unit 1)
-				)
-			)
-		)
-	)
-	(symbol
-		(lib_id "Connector_Generic:Conn_02x20_Odd_Even")
+					(reference "R803")
+					(unit 1)
+				)
+			)
+		)
+	)
+	(symbol
+		(lib_id "SensorBoards:PiZero")
 		(at 180.34 66.04 0)
 		(unit 1)
@@
 		(dnp no)
 		(fields_autoplaced yes)
-		(property "Reference" "J16"
+		(property "Reference" "J801"
 			(at 181.61 36.83 0)
 			(effects
@@
 			)
 		)
-		(property "Value" "Conn_02x20_Odd_Even"
+		(property "Value" "PiZero"
 			(at 181.61 39.37 0)
 			(effects
@@
 			)
 		)
-		(property "Footprint" "Connector_PinHeader_1.27mm:PinHeader_2x20_P1.27mm_Horizontal"
+		(property "Footprint" "Module:Raspberry_Pi_Zero_Socketed_THT_FaceDown_MountingHoles"
 			(at 180.34 66.04 0)
 			(effects
@@
 			(project ""
 				(path "/278cfa6b-9496-4a22-b425-8abdb96793ef/1f6da6ca-ffaf-4729-a842-c849ecc1a6dc"
-					(reference "J16")
+					(reference "J801")
 					(unit 1)
 				)
@@
 		(dnp no)
 		(fields_autoplaced yes)
-		(property "Reference" "#PWR036"
+		(property "Reference" "#PWR0801"
 			(at 63.5 48.26 0)
 			(effects
@@
 			(project ""
 				(path "/278cfa6b-9496-4a22-b425-8abdb96793ef/1f6da6ca-ffaf-4729-a842-c849ecc1a6dc"
-					(reference "#PWR036")
+					(reference "#PWR0801")
 					(unit 1)
 				)
@@
 		(dnp no)
 		(fields_autoplaced yes)
-		(property "Reference" "R50"
+		(property "Reference" "R801"
 			(at 44.45 46.99 90)
 			(effects
@@
 			)
 		)
-		(property "Footprint" "Resistor_SMD:R_0815_2038Metric"
+		(property "Footprint" "Resistor_SMD:R_0805_2012Metric"
 			(at 44.45 55.118 90)
 			(effects
@@
 			(project ""
 				(path "/278cfa6b-9496-4a22-b425-8abdb96793ef/1f6da6ca-ffaf-4729-a842-c849ecc1a6dc"
-					(reference "R50")
+					(reference "R801")
 					(unit 1)
 				)
@@
 		(dnp no)
 		(fields_autoplaced yes)
-		(property "Reference" "K1"
+		(property "Reference" "K801"
 			(at 80.01 73.6599 0)
 			(effects
@@
 			(project ""
 				(path "/278cfa6b-9496-4a22-b425-8abdb96793ef/1f6da6ca-ffaf-4729-a842-c849ecc1a6dc"
-					(reference "K1")
+					(reference "K801")
 					(unit 1)
 				)
@@
 		(dnp no)
 		(fields_autoplaced yes)
-		(property "Reference" "R52"
+		(property "Reference" "R805"
 			(at 162.56 39.37 90)
 			(effects
@@
 			)
 		)
-		(property "Footprint" "Resistor_SMD:R_0815_2038Metric"
+		(property "Footprint" "Resistor_SMD:R_0805_2012Metric"
 			(at 162.56 43.942 90)
 			(effects
@@
 			(project ""
 				(path "/278cfa6b-9496-4a22-b425-8abdb96793ef/1f6da6ca-ffaf-4729-a842-c849ecc1a6dc"
-					(reference "R52")
+					(reference "R805")
 					(unit 1)
 				)
@@
 		(dnp no)
 		(fields_autoplaced yes)
-		(property "Reference" "#PWR034"
+		(property "Reference" "#PWR0804"
 			(at 173.99 100.33 0)
 			(effects
@@
 			(project ""
 				(path "/278cfa6b-9496-4a22-b425-8abdb96793ef/1f6da6ca-ffaf-4729-a842-c849ecc1a6dc"
-					(reference "#PWR034")
+					(reference "#PWR0804")
 					(unit 1)
 				)
@@
 		(dnp no)
 		(fields_autoplaced yes)
-		(property "Reference" "#PWR032"
+		(property "Reference" "#PWR0802"
 			(at 63.5 97.79 0)
 			(effects
@@
 			(project ""
 				(path "/278cfa6b-9496-4a22-b425-8abdb96793ef/1f6da6ca-ffaf-4729-a842-c849ecc1a6dc"
-					(reference "#PWR032")
+					(reference "#PWR0802")
 					(unit 1)
 				)
@@
 		(on_board yes)
 		(dnp no)
-		(property "Reference" "Q5"
+		(property "Reference" "Q801"
 			(at 66.04 52.0699 0)
 			(effects
@@
 			(project ""
 				(path "/278cfa6b-9496-4a22-b425-8abdb96793ef/1f6da6ca-ffaf-4729-a842-c849ecc1a6dc"
-					(reference "Q5")
+					(reference "Q801")
 					(unit 1)
 				)
@@
 		(dnp no)
 		(fields_autoplaced yes)
-		(property "Reference" "D4"
+		(property "Reference" "D801"
 			(at 53.34 73.6599 90)
 			(effects
@@
 			(project ""
 				(path "/278cfa6b-9496-4a22-b425-8abdb96793ef/1f6da6ca-ffaf-4729-a842-c849ecc1a6dc"
-					(reference "D4")
+					(reference "D801")
 					(unit 1)
 				)
@@
 		(dnp no)
 		(fields_autoplaced yes)
-		(property "Reference" "#PWR035"
+		(property "Reference" "#PWR0803"
 			(at 153.67 95.25 0)
 			(effects
@@
 			(project ""
 				(path "/278cfa6b-9496-4a22-b425-8abdb96793ef/1f6da6ca-ffaf-4729-a842-c849ecc1a6dc"
-					(reference "#PWR035")
+					(reference "#PWR0803")
 					(unit 1)
 				)
@@
 		(dnp no)
 		(fields_autoplaced yes)
-		(property "Reference" "R53"
+		(property "Reference" "R804"
 			(at 156.21 41.91 90)
 			(effects
@@
 			)
 		)
-		(property "Footprint" "Resistor_SMD:R_0815_2038Metric"
+		(property "Footprint" "Resistor_SMD:R_0805_2012Metric"
 			(at 156.21 50.038 90)
 			(effects
@@
 			(project ""
 				(path "/278cfa6b-9496-4a22-b425-8abdb96793ef/1f6da6ca-ffaf-4729-a842-c849ecc1a6dc"
-					(reference "R53")
-					(unit 1)
-				)
+					(reference "R804")
+					(unit 1)
+				)

Commit message: PCB and footprint arrangements
Parts:
- J801: footprint Module:Raspberry_Pi_Zero_Socketed_THT_FaceDown_MountingHoles -> SensorBoards:Raspberry_Pi_Zero_Socket_wo_drills
Changed lines of the file:
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@@
 			)
 		)
-		(property "Footprint" "Module:Raspberry_Pi_Zero_Socketed_THT_FaceDown_MountingHoles"
+		(property "Footprint" "SensorBoards:Raspberry_Pi_Zero_Socket_wo_drills"
 			(at 180.34 66.04 0)
 			(effects

Commit message: drawed a lot of things
Parts:
- added R703: 0, Resistor_SMD:R_0805_2012Metric, symbol Device:R
- renumbered D801 to D701, J801 to J701, K801 to K701, Q801 to Q701, R801 to R701, R802 to R702, R804 to R704, R803 to R705, R805 to R706
Connections:
- net READY: now also R703.1; no longer J701.29 (Pin_29), R705.1
- new net: J701.29 (Pin_29), R703.2, R705.1
Other:
- moved on the sheet: R705
Changed lines of the file:
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@@
 	)
 	(junction
-		(at 153.67 78.74)
+		(at 63.5 63.5)
 		(diameter 0)
 		(color 0 0 0 0)
 	)
 	(junction
-		(at 63.5 63.5)
+		(at 173.99 91.44)
 		(diameter 0)
 		(color 0 0 0 0)
 	)
 	(junction
-		(at 173.99 91.44)
+		(at 173.99 73.66)
 		(diameter 0)
 		(color 0 0 0 0)
 	)
 	(junction
-		(at 173.99 73.66)
+		(at 158.75 78.74)
 		(diameter 0)
 		(color 0 0 0 0)
@@
 	(wire
 		(pts
-			(xy 189.23 66.04) (xy 189.23 78.74)
+			(xy 158.75 78.74) (xy 158.75 82.55)
 		)
 		(stroke
@@
 	(wire
 		(pts
-			(xy 187.96 78.74) (xy 189.23 78.74)
+			(xy 189.23 66.04) (xy 189.23 78.74)
 		)
 		(stroke
@@
 	(wire
 		(pts
-			(xy 63.5 63.5) (xy 63.5 67.31)
+			(xy 187.96 78.74) (xy 189.23 78.74)
 		)
 		(stroke
@@
 	(wire
 		(pts
-			(xy 189.23 48.26) (xy 189.23 58.42)
+			(xy 63.5 63.5) (xy 63.5 67.31)
 		)
 		(stroke
@@
 	(wire
 		(pts
-			(xy 50.8 78.74) (xy 50.8 86.36)
+			(xy 189.23 48.26) (xy 189.23 58.42)
 		)
 		(stroke
@@
 	(wire
 		(pts
-			(xy 63.5 82.55) (xy 63.5 86.36)
+			(xy 50.8 78.74) (xy 50.8 86.36)
 		)
 		(stroke
@@
 	(wire
 		(pts
-			(xy 153.67 78.74) (xy 175.26 78.74)
+			(xy 63.5 82.55) (xy 63.5 86.36)
 		)
 		(stroke
@@
 	(wire
 		(pts
-			(xy 140.97 78.74) (xy 153.67 78.74)
+			(xy 140.97 78.74) (xy 144.78 78.74)
 		)
 		(stroke
@@
 	(wire
 		(pts
+			(xy 158.75 78.74) (xy 175.26 78.74)
+		)
+		(stroke
+			(width 0)
+			(type default)
+		)
+	)
+	(wire
+		(pts
 			(xy 73.66 82.55) (xy 73.66 91.44)
 		)
@@
 	(wire
 		(pts
-			(xy 173.99 91.44) (xy 175.26 91.44)
+			(xy 152.4 78.74) (xy 158.75 78.74)
 		)
 		(stroke
@@
 	(wire
 		(pts
-			(xy 189.23 45.72) (xy 189.23 43.18)
+			(xy 173.99 91.44) (xy 175.26 91.44)
 		)
 		(stroke
@@
 	(wire
 		(pts
-			(xy 76.2 54.61) (xy 76.2 44.45)
+			(xy 189.23 45.72) (xy 189.23 43.18)
 		)
 		(stroke
@@
 	(wire
 		(pts
-			(xy 175.26 73.66) (xy 173.99 73.66)
+			(xy 76.2 54.61) (xy 76.2 44.45)
 		)
 		(stroke
@@
 	(wire
 		(pts
-			(xy 189.23 33.02) (xy 189.23 43.18)
+			(xy 175.26 73.66) (xy 173.99 73.66)
 		)
 		(stroke
@@
 	(wire
 		(pts
-			(xy 153.67 78.74) (xy 153.67 81.28)
+			(xy 189.23 33.02) (xy 189.23 43.18)
 		)
 		(stroke
@@
 	(text "Software on Pi should configure this pin as OUTPUT.\n- set to HIGH when boot is finished.\n- set to LOW, when Zero can be powered down again."
 		(exclude_from_sim no)
-		(at 116.586 74.168 0)
+		(at 118.364 73.66 0)
 		(effects
 			(font
@@
 	(symbol
 		(lib_id "Device:R")
+		(at 148.59 78.74 90)
+		(unit 1)
+		(exclude_from_sim no)
+		(in_bom yes)
+		(on_board yes)
+		(dnp no)
+		(property "Reference" "R703"
+			(at 148.59 81.788 90)
+			(effects
+				(font
+					(size 1.27 1.27)
+				)
+			)
+		)
+		(property "Value" "0"
+			(at 148.59 84.328 90)
+			(effects
+				(font
+					(size 1.27 1.27)
+				)
+			)
+		)
+		(property "Footprint" "Resistor_SMD:R_0805_2012Metric"
+			(at 148.59 80.518 90)
+			(effects
+				(font
+					(size 1.27 1.27)
+				)
+				(hide yes)
+			)
+		)
+		(property "Datasheet" "~"
+			(at 148.59 78.74 0)
+			(effects
+				(font
+					(size 1.27 1.27)
+				)
+				(hide yes)
+			)
+		)
+		(property "Description" "Resistor"
+			(at 148.59 78.74 0)
+			(effects
+				(font
+					(size 1.27 1.27)
+				)
+				(hide yes)
+			)
+		)
+		(pin "2"
+		)
+		(pin "1"
+		)
+		(instances
+			(project ""
+				(path "/278cfa6b-9496-4a22-b425-8abdb96793ef/1f6da6ca-ffaf-4729-a842-c849ecc1a6dc"
+					(reference "R703")
+					(unit 1)
+				)
+			)
+		)
+	)
+	(symbol
+		(lib_id "Device:R")
 		(at 76.2 58.42 180)
 		(unit 1)
@@
 		(dnp no)
 		(fields_autoplaced yes)
-		(property "Reference" "R802"
+		(property "Reference" "R702"
 			(at 78.74 57.1499 0)
 			(effects
@@
 			(project ""
 				(path "/278cfa6b-9496-4a22-b425-8abdb96793ef/1f6da6ca-ffaf-4729-a842-c849ecc1a6dc"
-					(reference "R802")
+					(reference "R702")
 					(unit 1)
 				)
@@
 	(symbol
 		(lib_id "Device:R")
-		(at 153.67 85.09 0)
+		(at 158.75 86.36 0)
 		(unit 1)
 		(exclude_from_sim no)
@@
 		(dnp no)
 		(fields_autoplaced yes)
-		(property "Reference" "R803"
-			(at 156.21 83.8199 0)
+		(property "Reference" "R705"
+			(at 161.29 85.0899 0)
 			(effects
 				(font
@@
 		)
 		(property "Value" "4k7"
-			(at 156.21 86.3599 0)
+			(at 161.29 87.6299 0)
 			(effects
 				(font
@@
 		)
 		(property "Footprint" "Resistor_SMD:R_0805_2012Metric"
-			(at 151.892 85.09 90)
+			(at 156.972 86.36 90)
 			(effects
 				(font
@@
 		)
 		(property "Datasheet" "~"
-			(at 153.67 85.09 0)
+			(at 158.75 86.36 0)
 			(effects
 				(font
@@
 		)
 		(property "Description" "Resistor"
-			(at 153.67 85.09 0)
+			(at 158.75 86.36 0)
 			(effects
 				(font
@@
 			(project ""
 				(path "/278cfa6b-9496-4a22-b425-8abdb96793ef/1f6da6ca-ffaf-4729-a842-c849ecc1a6dc"
-					(reference "R803")
+					(reference "R705")
 					(unit 1)
 				)
@@
 		(dnp no)
 		(fields_autoplaced yes)
-		(property "Reference" "J801"
+		(property "Reference" "J701"
 			(at 181.61 36.83 0)
 			(effects
@@
 			(project ""
 				(path "/278cfa6b-9496-4a22-b425-8abdb96793ef/1f6da6ca-ffaf-4729-a842-c849ecc1a6dc"
-					(reference "J801")
+					(reference "J701")
 					(unit 1)
 				)
@@
 		(dnp no)
 		(fields_autoplaced yes)
-		(property "Reference" "#PWR0801"
+		(property "Reference" "#PWR0701"
 			(at 63.5 48.26 0)
 			(effects
@@
 			(project ""
 				(path "/278cfa6b-9496-4a22-b425-8abdb96793ef/1f6da6ca-ffaf-4729-a842-c849ecc1a6dc"
-					(reference "#PWR0801")
+					(reference "#PWR0701")
 					(unit 1)
 				)
@@
 		(dnp no)
 		(fields_autoplaced yes)
-		(property "Reference" "R801"
+		(property "Reference" "R701"
 			(at 44.45 46.99 90)
 			(effects
@@
 			(project ""
 				(path "/278cfa6b-9496-4a22-b425-8abdb96793ef/1f6da6ca-ffaf-4729-a842-c849ecc1a6dc"
-					(reference "R801")
+					(reference "R701")
 					(unit 1)
 				)
@@
 		(dnp no)
 		(fields_autoplaced yes)
-		(property "Reference" "K801"
+		(property "Reference" "K701"
 			(at 80.01 73.6599 0)
 			(effects
@@
 			(project ""
 				(path "/278cfa6b-9496-4a22-b425-8abdb96793ef/1f6da6ca-ffaf-4729-a842-c849ecc1a6dc"
-					(reference "K801")
+					(reference "K701")
 					(unit 1)
 				)
@@
 		(dnp no)
 		(fields_autoplaced yes)
-		(property "Reference" "R805"
+		(property "Reference" "R706"
 			(at 162.56 39.37 90)
 			(effects
@@
 			(project ""
 				(path "/278cfa6b-9496-4a22-b425-8abdb96793ef/1f6da6ca-ffaf-4729-a842-c849ecc1a6dc"
-					(reference "R805")
+					(reference "R706")
 					(unit 1)
 				)
@@
 		(dnp no)
 		(fields_autoplaced yes)
-		(property "Reference" "#PWR0804"
+		(property "Reference" "#PWR0704"
 			(at 173.99 100.33 0)
 			(effects
@@
 			(project ""
 				(path "/278cfa6b-9496-4a22-b425-8abdb96793ef/1f6da6ca-ffaf-4729-a842-c849ecc1a6dc"
-					(reference "#PWR0804")
+					(reference "#PWR0704")
 					(unit 1)
 				)
@@
 		(dnp no)
 		(fields_autoplaced yes)
-		(property "Reference" "#PWR0802"
+		(property "Reference" "#PWR0702"
 			(at 63.5 97.79 0)
 			(effects
@@
 			(project ""
 				(path "/278cfa6b-9496-4a22-b425-8abdb96793ef/1f6da6ca-ffaf-4729-a842-c849ecc1a6dc"
-					(reference "#PWR0802")
+					(reference "#PWR0702")
 					(unit 1)
 				)
@@
 		(on_board yes)
 		(dnp no)
-		(property "Reference" "Q801"
+		(property "Reference" "Q701"
 			(at 66.04 52.0699 0)
 			(effects
@@
 			(project ""
 				(path "/278cfa6b-9496-4a22-b425-8abdb96793ef/1f6da6ca-ffaf-4729-a842-c849ecc1a6dc"
-					(reference "Q801")
+					(reference "Q701")
 					(unit 1)
 				)
@@
 		(dnp no)
 		(fields_autoplaced yes)
-		(property "Reference" "D801"
+		(property "Reference" "D701"
 			(at 53.34 73.6599 90)
 			(effects
@@
 			(project ""
 				(path "/278cfa6b-9496-4a22-b425-8abdb96793ef/1f6da6ca-ffaf-4729-a842-c849ecc1a6dc"
-					(reference "D801")
+					(reference "D701")
 					(unit 1)
 				)
@@
 	(symbol
 		(lib_id "power:GND")
-		(at 153.67 88.9 0)
+		(at 158.75 90.17 0)
 		(unit 1)
 		(exclude_from_sim no)
@@
 		(dnp no)
 		(fields_autoplaced yes)
-		(property "Reference" "#PWR0803"
-			(at 153.67 95.25 0)
+		(property "Reference" "#PWR0703"
+			(at 158.75 96.52 0)
 			(effects
 				(font
@@
 		)
 		(property "Value" "GND"
-			(at 153.67 93.98 0)
+			(at 158.75 95.25 0)
 			(effects
 				(font
@@
 		)
 		(property "Footprint" ""
-			(at 153.67 88.9 0)
+			(at 158.75 90.17 0)
 			(effects
 				(font
@@
 		)
 		(property "Datasheet" ""
-			(at 153.67 88.9 0)
+			(at 158.75 90.17 0)
 			(effects
 				(font
@@
 		)
 		(property "Description" "Power symbol creates a global label with name \"GND\" , ground"
-			(at 153.67 88.9 0)
+			(at 158.75 90.17 0)
 			(effects
 				(font
@@
 			(project ""
 				(path "/278cfa6b-9496-4a22-b425-8abdb96793ef/1f6da6ca-ffaf-4729-a842-c849ecc1a6dc"
-					(reference "#PWR0803")
+					(reference "#PWR0703")
 					(unit 1)
 				)
@@
 		(dnp no)
 		(fields_autoplaced yes)
-		(property "Reference" "R804"
+		(property "Reference" "R704"
 			(at 156.21 41.91 90)
 			(effects
@@
 			(project ""
 				(path "/278cfa6b-9496-4a22-b425-8abdb96793ef/1f6da6ca-ffaf-4729-a842-c849ecc1a6dc"
-					(reference "R804")
+					(reference "R704")
 					(unit 1)
 				)

Commit message: added VCC-battery measurement line
Parts:
- Q701: MPN_Eurocircuit (none) -> MMBT3906
- R701: LCSC (none) -> C17415; MPN_Eurocircuit (none) -> GPR080510R
- R702, R703, R704, R706: LCSC (none) -> C17477; MPN_Eurocircuit (none) -> GPR08050R
- R705: LCSC (none) -> C17673; MPN_Eurocircuit (none) -> GPR08054K7
Changed lines of the file:
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@@
+			)
+		)
+		(property "LCSC" "C17477"
+			(at 148.59 78.74 0)
+			(effects
+				(font
+					(size 1.27 1.27)
+				)
+				(hide yes)
+			)
+		)
+		(property "MPN_Eurocircuit" "GPR08050R"
+			(at 148.59 78.74 0)
+			(effects
+				(font
+					(size 1.27 1.27)
+				)
+				(hide yes)
 			)
 		)
@@
 			)
 		)
+		(property "LCSC" "C17477"
+			(at 76.2 58.42 0)
+			(effects
+				(font
+					(size 1.27 1.27)
+				)
+				(hide yes)
+			)
+		)
+		(property "MPN_Eurocircuit" "GPR08050R"
+			(at 76.2 58.42 0)
+			(effects
+				(font
+					(size 1.27 1.27)
+				)
+				(hide yes)
+			)
+		)
 		(pin "2"
 		)
@@
 			)
 		)
+		(property "LCSC" "C17673"
+			(at 158.75 86.36 0)
+			(effects
+				(font
+					(size 1.27 1.27)
+				)
+				(hide yes)
+			)
+		)
+		(property "MPN_Eurocircuit" "GPR08054K7"
+			(at 158.75 86.36 0)
+			(effects
+				(font
+					(size 1.27 1.27)
+				)
+				(hide yes)
+			)
+		)
 		(pin "1"
 		)
@@
 			)
 		)
+		(property "MPN_Eurocircuit" ""
+			(at 180.34 66.04 0)
+			(effects
+				(font
+					(size 1.27 1.27)
+				)
+				(hide yes)
+			)
+		)
 		(pin "33"
 		)
@@
 			)
 		)
+		(property "LCSC" "C17415"
+			(at 44.45 53.34 0)
+			(effects
+				(font
+					(size 1.27 1.27)
+				)
+				(hide yes)
+			)
+		)
+		(property "MPN_Eurocircuit" "GPR080510R"
+			(at 44.45 53.34 0)
+			(effects
+				(font
+					(size 1.27 1.27)
+				)
+				(hide yes)
+			)
+		)
 		(pin "1"
 		)
@@
 			)
 		)
+		(property "MPN_Eurocircuit" ""
+			(at 68.58 74.93 0)
+			(effects
+				(font
+					(size 1.27 1.27)
+				)
+				(hide yes)
+			)
+		)
 		(pin "11"
 		)
@@
 		)
 		(property "Description" "Resistor"
+			(at 162.56 45.72 0)
+			(effects
+				(font
+					(size 1.27 1.27)
+				)
+				(hide yes)
+			)
+		)
+		(property "LCSC" "C17477"
+			(at 162.56 45.72 0)
+			(effects
+				(font
+					(size 1.27 1.27)
+				)
+				(hide yes)
+			)
+		)
+		(property "MPN_Eurocircuit" "GPR08050R"
 			(at 162.56 45.72 0)
 			(effects
@@
 			)
 		)
+		(property "MPN_Eurocircuit" "MMBT3906"
+			(at 60.96 53.34 0)
+			(effects
+				(font
+					(size 1.27 1.27)
+				)
+				(hide yes)
+			)
+		)
 		(pin "1"
 		)
@@
 			)
 		)
+		(property "MPN_Eurocircuit" ""
+			(at 50.8 74.93 0)
+			(effects
+				(font
+					(size 1.27 1.27)
+				)
+				(hide yes)
+			)
+		)
 		(pin "1"
 		)
@@
 			(at 156.21 48.26 0)
 			(effects
+				(font
+					(size 1.27 1.27)
+				)
+				(hide yes)
+			)
+		)
+		(property "LCSC" "C17477"
+			(at 156.21 48.26 0)
+			(effects
+				(font
+					(size 1.27 1.27)
+				)
+				(hide yes)
+			)
+		)
+		(property "MPN_Eurocircuit" "GPR08050R"
+			(at 156.21 48.26 0)
+			(effects

Commit message: rev1
Parts:
- D701, Q701: OrderStatus (none) -> order
- J701, K701: OrderStatus (none) -> manual
- R701, R702, R703, R704, R705, R706: OrderStatus (none) -> assembly
Changed lines of the file:
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@@
+			)
+		)
+		(property "OrderStatus" "assembly"
+			(at 148.59 78.74 0)
+			(effects
+				(font
+					(size 1.27 1.27)
+				)
+				(hide yes)
 			)
 		)
@@
 			)
 		)
+		(property "OrderStatus" "assembly"
+			(at 76.2 58.42 0)
+			(effects
+				(font
+					(size 1.27 1.27)
+				)
+				(hide yes)
+			)
+		)
 		(pin "2"
 		)
@@
 			)
 		)
+		(property "OrderStatus" "assembly"
+			(at 158.75 86.36 0)
+			(effects
+				(font
+					(size 1.27 1.27)
+				)
+				(hide yes)
+			)
+		)
 		(pin "1"
 		)
@@
 			)
 		)
+		(property "OrderStatus" "manual"
+			(at 180.34 66.04 0)
+			(effects
+				(font
+					(size 1.27 1.27)
+				)
+				(hide yes)
+			)
+		)
 		(pin "33"
 		)
@@
 			)
 		)
+		(property "OrderStatus" "assembly"
+			(at 44.45 53.34 0)
+			(effects
+				(font
+					(size 1.27 1.27)
+				)
+				(hide yes)
+			)
+		)
 		(pin "1"
 		)
@@
 			)
 		)
+		(property "OrderStatus" "manual"
+			(at 68.58 74.93 0)
+			(effects
+				(font
+					(size 1.27 1.27)
+				)
+				(hide yes)
+			)
+		)
 		(pin "11"
 		)
@@
 			)
 		)
+		(property "OrderStatus" "assembly"
+			(at 162.56 45.72 0)
+			(effects
+				(font
+					(size 1.27 1.27)
+				)
+				(hide yes)
+			)
+		)
 		(pin "1"
 		)
@@
 			)
 		)
+		(property "OrderStatus" "order"
+			(at 60.96 53.34 0)
+			(effects
+				(font
+					(size 1.27 1.27)
+				)
+				(hide yes)
+			)
+		)
 		(pin "1"
 		)
@@
 			)
 		)
+		(property "OrderStatus" "order"
+			(at 50.8 74.93 0)
+			(effects
+				(font
+					(size 1.27 1.27)
+				)
+				(hide yes)
+			)
+		)
 		(pin "1"
 		)
@@
 			(at 156.21 48.26 0)
 			(effects
+				(font
+					(size 1.27 1.27)
+				)
+				(hide yes)
+			)
+		)
+		(property "OrderStatus" "assembly"
+			(at 156.21 48.26 0)
+			(effects
