File: pouch2/sd_card.kicad_sch (KiCad schematic)
At the start: 1 part

Commit message: started PCB design
Parts:
- U401: renamed from U4; footprint (none) -> Connector_PinHeader_2.54mm:PinHeader_1x06_P2.54mm_Vertical
Changed lines of the file:
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@@
 		(dnp no)
 		(fields_autoplaced yes)
-		(property "Reference" "U4"
+		(property "Reference" "U401"
 			(at 123.19 85.7249 0)
 			(effects
@@
 			)
 		)
-		(property "Footprint" ""
+		(property "Footprint" "Connector_PinHeader_2.54mm:PinHeader_1x06_P2.54mm_Vertical"
 			(at 132.08 97.79 0)
 			(effects
@@
 			(project ""
 				(path "/278cfa6b-9496-4a22-b425-8abdb96793ef/4c18d891-44a5-41ab-9141-17f4525bee9f"
-					(reference "U4")
+					(reference "U401")
 					(unit 1)
 				)
@@
 		(dnp no)
 		(fields_autoplaced yes)
-		(property "Reference" "#PWR016"
+		(property "Reference" "#PWR0401"
 			(at 130.81 114.3 0)
 			(effects
@@
 			(project ""
 				(path "/278cfa6b-9496-4a22-b425-8abdb96793ef/4c18d891-44a5-41ab-9141-17f4525bee9f"
-					(reference "#PWR016")
+					(reference "#PWR0401")
 					(unit 1)
 				)

Commit message: updated backside of PCB
Parts:
- U401: footprint Connector_PinHeader_2.54mm:PinHeader_1x06_P2.54mm_Vertical -> SensorBoards:DEBO_SD-Card
Changed lines of the file:
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@@
 			)
 		)
-		(property "Footprint" "Connector_PinHeader_2.54mm:PinHeader_1x06_P2.54mm_Vertical"
+		(property "Footprint" "SensorBoards:DEBO_SD-Card"
 			(at 132.08 97.79 0)
 			(effects

Commit message: started routing
Parts:
- added R401, R402, R403, R404: 0, Resistor_SMD:R_0805_2012Metric, symbol Device:R
Connections:
- net CS: now also R404.1; no longer U401.6 (CS)
- net MISO: now also R401.2; no longer U401.3 (MISO)
- net MOSI: now also R402.1; no longer U401.4 (MOSI)
- net SCK: now also R403.2; no longer U401.5 (SCK)
- new net: R402.2, U401.4 (MOSI)
- new net: R404.2, U401.6 (CS)
- new net: R403.1, U401.5 (SCK)
- new net: R401.1, U401.3 (MISO)

Commit message: drawed a lot of things
Parts:
- renumbered R403 to R402, R402 to R403
Changed lines of the file:
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@@
 		(on_board yes)
 		(dnp no)
-		(property "Reference" "R402"
+		(property "Reference" "R403"
 			(at 151.13 83.058 90)
 			(effects
@@
 			(project ""
 				(path "/278cfa6b-9496-4a22-b425-8abdb96793ef/4c18d891-44a5-41ab-9141-17f4525bee9f"
-					(reference "R402")
+					(reference "R403")
 					(unit 1)
 				)
@@
 		(on_board yes)
 		(dnp no)
-		(property "Reference" "R403"
+		(property "Reference" "R402"
 			(at 143.256 89.916 90)
 			(effects
@@
 			(project ""
 				(path "/278cfa6b-9496-4a22-b425-8abdb96793ef/4c18d891-44a5-41ab-9141-17f4525bee9f"
-					(reference "R403")
+					(reference "R402")
 					(unit 1)
 				)

Commit message: added VCC-battery measurement line
Parts:
- R401, R402, R403, R404: LCSC (none) -> C17477; MPN_Eurocircuit (none) -> GPR08050R
Changed lines of the file:
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@@
+			)
+		)
+		(property "LCSC" "C17477"
+			(at 151.13 85.09 0)
+			(effects
+				(font
+					(size 1.27 1.27)
+				)
+				(hide yes)
+			)
+		)
+		(property "MPN_Eurocircuit" "GPR08050R"
+			(at 151.13 85.09 0)
+			(effects
+				(font
+					(size 1.27 1.27)
+				)
+				(hide yes)
 			)
 		)
@@
 			)
 		)
+		(property "LCSC" "C17477"
+			(at 151.13 90.17 0)
+			(effects
+				(font
+					(size 1.27 1.27)
+				)
+				(hide yes)
+			)
+		)
+		(property "MPN_Eurocircuit" "GPR08050R"
+			(at 151.13 90.17 0)
+			(effects
+				(font
+					(size 1.27 1.27)
+				)
+				(hide yes)
+			)
+		)
 		(pin "1"
 		)
@@
 		)
 		(property "Description" "Resistor"
+			(at 143.51 87.63 0)
+			(effects
+				(font
+					(size 1.27 1.27)
+				)
+				(hide yes)
+			)
+		)
+		(property "LCSC" "C17477"
+			(at 143.51 87.63 0)
+			(effects
+				(font
+					(size 1.27 1.27)
+				)
+				(hide yes)
+			)
+		)
+		(property "MPN_Eurocircuit" "GPR08050R"
 			(at 143.51 87.63 0)
 			(effects
@@
 			)
 		)
+		(property "MPN_Eurocircuit" ""
+			(at 132.08 97.79 0)
+			(effects
+				(font
+					(size 1.27 1.27)
+				)
+				(hide yes)
+			)
+		)
 		(pin "4"
 		)
@@
 			(at 143.51 82.55 0)
 			(effects
+				(font
+					(size 1.27 1.27)
+				)
+				(hide yes)
+			)
+		)
+		(property "LCSC" "C17477"
+			(at 143.51 82.55 0)
+			(effects
+				(font
+					(size 1.27 1.27)
+				)
+				(hide yes)
+			)
+		)
+		(property "MPN_Eurocircuit" "GPR08050R"
+			(at 143.51 82.55 0)
+			(effects

Commit message: rev1
Parts:
- R401, R402, R403, R404: OrderStatus (none) -> assembly
- U401: OrderStatus (none) -> manual
Changed lines of the file:
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@@
+			)
+		)
+		(property "OrderStatus" "assembly"
+			(at 151.13 85.09 0)
+			(effects
+				(font
+					(size 1.27 1.27)
+				)
+				(hide yes)
 			)
 		)
@@
 			)
 		)
+		(property "OrderStatus" "assembly"
+			(at 151.13 90.17 0)
+			(effects
+				(font
+					(size 1.27 1.27)
+				)
+				(hide yes)
+			)
+		)
 		(pin "1"
 		)
@@
 		)
 		(property "MPN_Eurocircuit" "GPR08050R"
+			(at 143.51 87.63 0)
+			(effects
+				(font
+					(size 1.27 1.27)
+				)
+				(hide yes)
+			)
+		)
+		(property "OrderStatus" "assembly"
 			(at 143.51 87.63 0)
 			(effects
@@
 			)
 		)
+		(property "OrderStatus" "manual"
+			(at 132.08 97.79 0)
+			(effects
+				(font
+					(size 1.27 1.27)
+				)
+				(hide yes)
+			)
+		)
 		(pin "4"
 		)
@@
 			(at 143.51 82.55 0)
 			(effects
+				(font
+					(size 1.27 1.27)
+				)
+				(hide yes)
+			)
+		)
+		(property "OrderStatus" "assembly"
+			(at 143.51 82.55 0)
+			(effects
